File: Sch/FX3_clk_reset_cn.sch (KiCad schematic (older format))
At the start: 21 parts, among them CN1 USB3_micro_B, IC1 CYUSB3014, SW1 DIP_SW_4POS, Y1 19.2MHz

Commit message: modify
Parts:
- added unit 5 of IC1
- added R13, R14: 10k, symbol R
- added RN1: 22, symbol R_Pack04
- R4: value 10k -> DNL
Connections:
- net labels added: FX3_CTL[15], FX3_RESET#, FX3_VIO1, FX3_VIO5
- net labels removed: VIO1
- wire segments 67 -> 74
Other:
- note added: "PMODE[2:0]=0F1:SPI->USB, F11:USB"
- moved on the sheet: R5, SW1
Changed lines of the file:
@@
 $EndDescr
 $Comp
-L GND #PWR4
+L GND #PWR01
 U 1 1 589AE25B
 P 4850 4200
-F 0 "#PWR4" H 4850 3950 50  0001 C CNN
+F 0 "#PWR01" H 4850 3950 50  0001 C CNN
 F 1 "GND" H 4850 4050 50  0000 C CNN
 F 2 "" H 4850 4200 50  0000 C CNN
@@
 $EndComp
 $Comp
-L GND #PWR3
+L GND #PWR02
 U 1 1 589AE268
 P 4550 4200
-F 0 "#PWR3" H 4550 3950 50  0001 C CNN
+F 0 "#PWR02" H 4550 3950 50  0001 C CNN
 F 1 "GND" H 4550 4050 50  0000 C CNN
 F 2 "" H 4550 4200 50  0000 C CNN
@@
 $EndComp
 $Comp
-L GND #PWR1
+L GND #PWR03
 U 1 1 589AE27C
 P 1350 3450
-F 0 "#PWR1" H 1350 3200 50  0001 C CNN
+F 0 "#PWR03" H 1350 3200 50  0001 C CNN
 F 1 "GND" H 1350 3300 50  0000 C CNN
 F 2 "" H 1350 3450 50  0000 C CNN
@@
 $EndComp
 $Comp
-L GND #PWR6
+L GND #PWR04
 U 1 1 589AEE63
 P 7250 4450
-F 0 "#PWR6" H 7250 4200 50  0001 C CNN
+F 0 "#PWR04" H 7250 4200 50  0001 C CNN
 F 1 "GND" H 7250 4300 50  0000 C CNN
 F 2 "" H 7250 4450 50  0000 C CNN
@@
 $EndComp
 $Comp
-L GND #PWR10
+L GND #PWR05
 U 1 1 58A053A3
 P 8700 4900
-F 0 "#PWR10" H 8700 4650 50  0001 C CNN
+F 0 "#PWR05" H 8700 4650 50  0001 C CNN
 F 1 "GND" H 8700 4750 50  0000 C CNN
 F 2 "" H 8700 4900 50  0000 C CNN
@@
 $EndComp
 $Comp
-L GND #PWR11
+L GND #PWR06
 U 1 1 58A0545F
 P 8950 4900
-F 0 "#PWR11" H 8950 4650 50  0001 C CNN
+F 0 "#PWR06" H 8950 4650 50  0001 C CNN
 F 1 "GND" H 8950 4750 50  0000 C CNN
 F 2 "" H 8950 4900 50  0000 C CNN
@@
 $EndComp
 $Comp
-L GND #PWR7
+L GND #PWR07
 U 1 1 58A05EBD
 P 7800 4900
-F 0 "#PWR7" H 7800 4650 50  0001 C CNN
+F 0 "#PWR07" H 7800 4650 50  0001 C CNN
 F 1 "GND" H 7800 4750 50  0000 C CNN
 F 2 "" H 7800 4900 50  0000 C CNN
@@
 $EndComp
 $Comp
-L GND #PWR8
+L GND #PWR08
 U 1 1 58A05EE5
 P 8000 4900
-F 0 "#PWR8" H 8000 4650 50  0001 C CNN
+F 0 "#PWR08" H 8000 4650 50  0001 C CNN
 F 1 "GND" H 8000 4750 50  0000 C CNN
 F 2 "" H 8000 4900 50  0000 C CNN
@@
 $EndComp
 $Comp
-L GND #PWR9
+L GND #PWR09
 U 1 1 58A06182
 P 8250 4900
-F 0 "#PWR9" H 8250 4650 50  0001 C CNN
+F 0 "#PWR09" H 8250 4650 50  0001 C CNN
 F 1 "GND" H 8250 4750 50  0000 C CNN
 F 2 "" H 8250 4900 50  0000 C CNN
@@
 $EndComp
 $Comp
-L GND #PWR5
+L GND #PWR010
 U 1 1 58A06620
 P 7000 4900
-F 0 "#PWR5" H 7000 4650 50  0001 C CNN
+F 0 "#PWR010" H 7000 4650 50  0001 C CNN
 F 1 "GND" H 7000 4750 50  0000 C CNN
 F 2 "" H 7000 4900 50  0000 C CNN
@@
 	7000 3100 7000 4600
 Wire Wire Line
-	3700 5900 4500 5900
-Text Label 3950 5900 0    60   ~ 0
-VIO1
+	2350 5900 4500 5900
 $Comp
 L R R4
@@
 P 4200 6050
 F 0 "R4" V 4280 6050 50  0000 C CNN
-F 1 "10k" V 4200 6050 50  0000 C CNN
+F 1 "DNL" V 4200 6050 50  0000 C CNN
 F 2 "" V 4130 6050 50  0000 C CNN
 F 3 "" H 4200 6050 50  0000 C CNN
@@
 L R R5
 U 1 1 58A07409
-P 4350 6050
-F 0 "R5" V 4430 6050 50  0000 C CNN
-F 1 "10k" V 4350 6050 50  0000 C CNN
-F 2 "" V 4280 6050 50  0000 C CNN
-F 3 "" H 4350 6050 50  0000 C CNN
-	1    4350 6050
+P 2550 6050
+F 0 "R5" V 2630 6050 50  0000 C CNN
+F 1 "10k" V 2550 6050 50  0000 C CNN
+F 2 "" V 2480 6050 50  0000 C CNN
+F 3 "" H 2550 6050 50  0000 C CNN
+	1    2550 6050
 	1    0    0    -1
 $EndComp
@@
 	1    0    0    -1
 $EndComp
-Connection ~ 4350 5900
 Wire Wire Line
 	4500 6200 4500 6450
@@
 	4000 6450 5050 6450
 Wire Wire Line
-	4350 6200 4350 6550
-Wire Wire Line
 	4000 6550 5050 6550
 Wire Wire Line
@@
 	4000 6650 5050 6650
 $Comp
-L GND #PWR2
+L GND #PWR011
 U 1 1 58A077E4
-P 3100 6850
-F 0 "#PWR2" H 3100 6600 50  0001 C CNN
-F 1 "GND" H 3100 6700 50  0000 C CNN
-F 2 "" H 3100 6850 50  0000 C CNN
-F 3 "" H 3100 6850 50  0000 C CNN
-	1    3100 6850
+P 2700 6850
+F 0 "#PWR011" H 2700 6600 50  0001 C CNN
+F 1 "GND" H 2700 6700 50  0000 C CNN
+F 2 "" H 2700 6850 50  0000 C CNN
+F 3 "" H 2700 6850 50  0000 C CNN
+	1    2700 6850
 	1    0    0    -1
 $EndComp
@@
 L DIP_SW_4POS SW1
 U 1 1 58A07985
-P 3650 6600
-F 0 "SW1" H 3650 6250 60  0000 C CNN
-F 1 "DIP_SW_4POS" H 3650 6950 60  0000 C CNN
-F 2 "" H 3750 6450 60  0001 C CNN
-F 3 "" H 3750 6450 60  0001 C CNN
-	1    3650 6600
-	1    0    0    -1
-$EndComp
-NoConn ~ 3300 6750
-Wire Wire Line
-	3300 6450 3100 6450
-Wire Wire Line
-	3100 6450 3100 6850
-Wire Wire Line
-	3300 6550 3100 6550
-Connection ~ 3100 6550
-Wire Wire Line
-	3300 6650 3100 6650
-Connection ~ 3100 6650
+P 3250 6600
+F 0 "SW1" H 3250 6250 60  0000 C CNN
+F 1 "DIP_SW_4POS" H 3250 6950 60  0000 C CNN
+F 2 "" H 3350 6450 60  0001 C CNN
+F 3 "" H 3350 6450 60  0001 C CNN
+	1    3250 6600
+	1    0    0    -1
+$EndComp
+NoConn ~ 2900 6750
+Wire Wire Line
+	2900 6450 2700 6450
+Wire Wire Line
+	2700 6450 2700 6850
+Wire Wire Line
+	2900 6650 2700 6650
+Connection ~ 2700 6650
 Connection ~ 4500 6450
-Connection ~ 4350 6550
 Connection ~ 4200 6650
+Wire Wire Line
+	5050 6750 4600 6750
+Wire Wire Line
+	4600 6750 4600 7350
+Wire Wire Line
+	4600 7350 2550 7350
+Text GLabel 4000 2950 2    60   Input ~ 0
+FX3_RESET#
+Text GLabel 2550 7350 0    60   Input ~ 0
+FX3_CTL[15]
+Text Notes 4900 6150 0    60   ~ 0
+PMODE[2:0]=0F1:SPI->USB, F11:USB
+$Comp
+L R_Pack04 RN1
+U 1 1 58A34597
+P 3800 6650
+F 0 "RN1" V 3500 6650 50  0000 C CNN
+F 1 "22" V 4000 6650 50  0000 C CNN
+F 2 "" V 4075 6650 50  0001 C CNN
+F 3 "" H 3800 6650 50  0000 C CNN
+	1    3800 6650
+	0    1    1    0
+$EndComp
 NoConn ~ 4000 6750
 Wire Wire Line
-	5050 6750 4600 6750
-Wire Wire Line
-	4600 6750 4600 7350
-Wire Wire Line
-	4600 7350 2550 7350
+	2900 6550 2550 6550
+Wire Wire Line
+	2550 6550 2550 6200
+$Comp
+L CYUSB3014 IC1
+U 5 1 58A3F3B9
+P 5650 1550
+F 0 "IC1" H 5650 -800 50  0000 C CNN
+F 1 "CYUSB3014" H 5650 4100 50  0000 C CNN
+F 2 "MODULE" H 5600 3850 50  0001 C CNN
+F 3 "DOCUMENTATION" H 5650 4000 50  0001 C CNN
+	5    5650 1550
+	1    0    0    -1
+$EndComp
+Text GLabel 4450 650  0    60   Input ~ 0
+FX3_VIO5
+$Comp
+L R R13
+U 1 1 58A3F7D9
+P 4600 900
+F 0 "R13" V 4680 900 50  0000 C CNN
+F 1 "10k" V 4600 900 50  0000 C CNN
+F 2 "" V 4530 900 50  0000 C CNN
+F 3 "" H 4600 900 50  0000 C CNN
+	1    4600 900
+	1    0    0    -1
+$EndComp
+$Comp
+L R R14
+U 1 1 58A3F8D8
+P 4750 900
+F 0 "R14" V 4830 900 50  0000 C CNN
+F 1 "10k" V 4750 900 50  0000 C CNN
+F 2 "" V 4680 900 50  0000 C CNN
+F 3 "" H 4750 900 50  0000 C CNN
+	1    4750 900
+	1    0    0    -1
+$EndComp
+Wire Wire Line
+	4450 650  4750 650
+Wire Wire Line
+	4600 650  4600 750
+Wire Wire Line
+	4750 650  4750 750
+Connection ~ 4600 650
+Wire Wire Line
+	4750 1050 4750 1150
+Wire Wire Line
+	4750 1150 4900 1150
+Wire Wire Line
+	4600 1050 4600 1250
+Wire Wire Line
+	4600 1250 4900 1250
+Text GLabel 2350 5900 0    60   Input ~ 0
+FX3_VIO1
+Connection ~ 4200 5900
+Connection ~ 2550 5900
 $EndSCHEMATC

Commit message: update
Parts:
- added C51, C52: C, symbol C
- added IC2: NCP361SNT1G, symbol NCP361SNT1G
- added L10: MPZ2012S601A, symbol L
- added P3: CONN_01X05, symbol CONN_01X05
- added R23: 1M, symbol R
- added RN12: 10k, Resistors_ThroughHole:Resistor_Array_SIP5, symbol R_Network04
- added W1: TEST_1P, symbol TEST_1P
Connections:
- net labels added: +3V3, USB_VBUS
- net labels removed: FX3_VIO1, FX3_VIO5
- wire segments 74 -> 96
Other:
- moved on the sheet: C1, C2, IC1D, IC1E, R1, R13, R14, R2, R3, Y1
