File: Sch/FX3VDD.sch (KiCad schematic (older format))
At the start: 10 parts, among them U3 TLV62130A

Commit message: modify
Parts:
- gave numbers to parts that had none: 1
Changed lines of the file:
@@
 $EndComp
 Wire Wire Line
-	3550 1800 3550 1950
-Wire Wire Line
-	3550 1950 3550 2150
-Wire Wire Line
-	3550 2450 3550 2550
-Wire Wire Line
-	3550 2550 3550 2650
-Wire Wire Line
-	3550 1950 4050 1950
-Wire Wire Line
-	4050 1950 4500 1950
-Wire Wire Line
-	4500 1950 4500 2150
-Wire Wire Line
-	4500 2150 4500 2250
-Wire Wire Line
-	4500 2250 4500 2350
-Wire Wire Line
-	4500 2350 4500 2550
+	3550 1800 3550 2150
+Wire Wire Line
+	3550 2450 3550 2650
+Wire Wire Line
+	3550 1950 4500 1950
+Wire Wire Line
+	4500 1950 4500 2550
 Connection ~ 3550 1950
 Wire Wire Line
@@
 	5250 3150 5250 3250
 Wire Wire Line
-	5250 3250 5350 3250
-Wire Wire Line
-	5350 3250 5450 3250
-Wire Wire Line
-	5450 3250 5550 3250
-Wire Wire Line
-	5550 3250 5750 3250
-Wire Wire Line
-	5750 3250 5850 3250
-Wire Wire Line
-	5850 3250 6050 3250
+	5250 3250 6050 3250
 Wire Wire Line
 	6050 3250 6050 3350
@@
 Connection ~ 5850 3250
 Wire Wire Line
-	6100 2350 6300 2350
-Wire Wire Line
-	6300 2350 6300 2250
-Wire Wire Line
-	6300 2250 6300 2150
-Wire Wire Line
-	6100 2150 6300 2150
-Wire Wire Line
-	6300 2150 6450 2150
+	6300 2350 6100 2350
+Wire Wire Line
+	6300 2150 6300 2350
+Wire Wire Line
+	6100 2150 6450 2150
 Wire Wire Line
 	6100 2250 6300 2250
@@
 Connection ~ 6300 2150
 Wire Wire Line
-	6750 2150 6950 2150
-Wire Wire Line
-	6950 2150 7200 2150
-Wire Wire Line
-	7200 2150 7600 2150
-Wire Wire Line
-	7600 2150 8150 2150
+	6750 2150 8150 2150
 Wire Wire Line
 	6950 2150 6950 2500
@@
 Connection ~ 6950 2150
 Wire Wire Line
-	6750 2600 6550 2600
-Wire Wire Line
-	6550 2600 6100 2600
+	6100 2600 6750 2600
 Wire Wire Line
 	6550 3050 6550 2600
@@
 $EndComp
 Wire Wire Line
-	6100 2700 9100 2700
-Wire Wire Line
-	9100 2700 9500 2700
+	6100 2700 9500 2700
 Wire Wire Line
 	9100 2700 9100 2450
@@
 PG_FX3VDD
 $Comp
-L C C?
+L C C57
 U 1 1 58A52E48
 P 4050 2300
-F 0 "C?" H 4075 2400 50  0000 L CNN
+F 0 "C57" H 4075 2400 50  0000 L CNN
 F 1 "0.1uF" H 4075 2200 50  0000 L CNN
 F 2 "" H 4088 2150 50  0000 C CNN
