File: Sch/adc/CN.sch (KiCad schematic (older format))
At the start: 15 parts, among them J1 JP4, J2 Header5, P1 CONN_02X40, U1 LTC2292

Commit message: Schematics done
Parts:
- added R12: 22, symbol R
- added RN5: 22, symbol R_Pack04
- added W1, W2: TEST_1P, symbol TEST_1P
- R1: renamed from R?; value 49k -> 10k
- gave numbers to parts that had none: 2
Connections:
- no-connect marks 57 -> 59
Changed lines of the file:
@@
 $EndComp
 $Comp
-L GND #PWR07
-U 1 1 58A4E278
-P 8650 900
-F 0 "#PWR07" H 8650 650 50  0001 C CNN
-F 1 "GND" H 8650 750 50  0000 C CNN
-F 2 "" H 8650 900 50  0000 C CNN
-F 3 "" H 8650 900 50  0000 C CNN
-	1    8650 900
-	1    0    0    -1
-$EndComp
-$Comp
-L PWR_FLAG #FLG08
-U 1 1 58A4E2AC
-P 8650 900
-F 0 "#FLG08" H 8650 995 50  0001 C CNN
-F 1 "PWR_FLAG" H 8650 1080 50  0000 C CNN
-F 2 "" H 8650 900 50  0000 C CNN
-F 3 "" H 8650 900 50  0000 C CNN
-	1    8650 900
-	1    0    0    -1
-$EndComp
-$Comp
-L PWR_FLAG #FLG09
+L PWR_FLAG #FLG07
 U 1 1 58A4E2FE
 P 8300 850
-F 0 "#FLG09" H 8300 945 50  0001 C CNN
+F 0 "#FLG07" H 8300 945 50  0001 C CNN
 F 1 "PWR_FLAG" H 8300 1030 50  0000 C CNN
 F 2 "" H 8300 850 50  0000 C CNN
@@
 $EndComp
 $Comp
-L PWR_FLAG #FLG010
+L PWR_FLAG #FLG08
 U 1 1 58A4E385
 P 7900 850
-F 0 "#FLG010" H 7900 945 50  0001 C CNN
+F 0 "#FLG08" H 7900 945 50  0001 C CNN
 F 1 "PWR_FLAG" H 7900 1030 50  0000 C CNN
 F 2 "" H 7900 850 50  0000 C CNN
@@
 $EndComp
 $Comp
-L GND #PWR011
+L GND #PWR09
 U 1 1 58A5EE0A
 P 3150 7100
-F 0 "#PWR011" H 3150 6850 50  0001 C CNN
+F 0 "#PWR09" H 3150 6850 50  0001 C CNN
 F 1 "GND" H 3150 6950 50  0000 C CNN
 F 2 "" H 3150 7100 50  0000 C CNN
@@
 VDD3
 $Comp
-L GND #PWR?
+L GND #PWR010
 U 1 1 58A86709
 P 950 2950
-F 0 "#PWR?" H 950 2700 50  0001 C CNN
+F 0 "#PWR010" H 950 2700 50  0001 C CNN
 F 1 "GND" H 950 2800 50  0000 C CNN
 F 2 "" H 950 2950 50  0000 C CNN
@@
 $EndComp
 $Comp
-L R R?
+L R R1
 U 1 1 58A86735
 P 950 2800
-F 0 "R?" V 1030 2800 50  0000 C CNN
-F 1 "49k" V 950 2800 50  0000 C CNN
+F 0 "R1" V 1030 2800 50  0000 C CNN
+F 1 "10k" V 950 2800 50  0000 C CNN
 F 2 "" V 880 2800 50  0000 C CNN
 F 3 "" H 950 2800 50  0000 C CNN
@@
 $EndComp
 $Comp
-L GND #PWR?
+L GND #PWR011
 U 1 1 58A87202
 P 1600 3350
-F 0 "#PWR?" H 1600 3100 50  0001 C CNN
+F 0 "#PWR011" H 1600 3100 50  0001 C CNN
 F 1 "GND" H 1600 3200 50  0000 C CNN
 F 2 "" H 1600 3350 50  0000 C CNN
@@
 $EndComp
 $Comp
-L R R?
+L R R10
 U 1 1 58A87208
 P 1600 3200
-F 0 "R?" V 1680 3200 50  0000 C CNN
+F 0 "R10" V 1680 3200 50  0000 C CNN
 F 1 "49k" V 1600 3200 50  0000 C CNN
 F 2 "" V 1530 3200 50  0000 C CNN
@@
 	7150 2450 7850 2450
 Wire Wire Line
-	7150 2550 7850 2550
-Wire Wire Line
-	7150 2650 7850 2650
-Wire Wire Line
-	7150 2750 7850 2750
+	7150 2550 8650 2550
+Wire Wire Line
+	7150 2650 8650 2650
+Wire Wire Line
+	7150 2750 8650 2750
 Wire Wire Line
 	7150 2950 7850 2950
@@
 	950  2600 950  2650
 $Comp
-L GND #PWR?
+L GND #PWR012
 U 1 1 58A87749
 P 1750 3350
-F 0 "#PWR?" H 1750 3100 50  0001 C CNN
+F 0 "#PWR012" H 1750 3100 50  0001 C CNN
 F 1 "GND" H 1750 3200 50  0000 C CNN
 F 2 "" H 1750 3350 50  0000 C CNN
@@
 $EndComp
 $Comp
-L R R?
+L R R11
 U 1 1 58A8774F
 P 1750 3200
-F 0 "R?" V 1830 3200 50  0000 C CNN
+F 0 "R11" V 1830 3200 50  0000 C CNN
 F 1 "49k" V 1750 3200 50  0000 C CNN
 F 2 "" V 1680 3200 50  0000 C CNN
@@
 Text Notes 750  3300 0    60   ~ 0
 High=nap mode
-Text GLabel 7850 2550 2    60   Output ~ 0
+Text GLabel 9050 2550 2    60   Output ~ 0
 FS
-Text GLabel 7850 2650 2    60   Output ~ 0
+Text GLabel 9050 2650 2    60   Output ~ 0
 BCLK
-Text GLabel 7850 2750 2    60   Output ~ 0
+Text GLabel 9050 2750 2    60   Output ~ 0
 DACIN
-Text GLabel 5950 4050 0    60   Output ~ 0
+Text GLabel 5650 4050 0    60   Output ~ 0
 MCLK
 Text GLabel 5950 2150 0    60   BiDi ~ 0
@@
 Text GLabel 5950 2250 0    60   BiDi ~ 0
 SDA
+$Comp
+L R_Pack04 RN5
+U 1 1 58A9A1DD
+P 8850 2650
+F 0 "RN5" V 8550 2650 50  0000 C CNN
+F 1 "22" V 9050 2650 50  0000 C CNN
+F 2 "" V 9125 2650 50  0001 C CNN
+F 3 "" H 8850 2650 50  0000 C CNN
+	1    8850 2650
+	0    1    1    0
+$EndComp
+NoConn ~ 8650 2450
+NoConn ~ 9050 2450
+$Comp
+L R R12
+U 1 1 58A9A823
+P 5800 4050
+F 0 "R12" V 5880 4050 50  0000 C CNN
+F 1 "22" V 5800 4050 50  0000 C CNN
+F 2 "" V 5730 4050 50  0000 C CNN
+F 3 "" H 5800 4050 50  0000 C CNN
+	1    5800 4050
+	0    -1   -1   0
+$EndComp
+$Comp
+L TEST_1P W1
+U 1 1 58A9D9D4
+P 5700 2450
+F 0 "W1" H 5700 2720 50  0000 C CNN
+F 1 "TEST_1P" H 5700 2650 50  0000 C CNN
+F 2 "" H 5900 2450 50  0000 C CNN
+F 3 "" H 5900 2450 50  0000 C CNN
+	1    5700 2450
+	0    -1   -1   0
+$EndComp
+$Comp
+L GND #PWR013
+U 1 1 58A9DDBA
+P 9850 1200
+F 0 "#PWR013" H 9850 950 50  0001 C CNN
+F 1 "GND" H 9850 1050 50  0000 C CNN
+F 2 "" H 9850 1200 50  0000 C CNN
+F 3 "" H 9850 1200 50  0000 C CNN
+	1    9850 1200
+	1    0    0    -1
+$EndComp
+$Comp
+L TEST_1P W2
+U 1 1 58A9DDF2
+P 9850 1200
+F 0 "W2" H 9850 1470 50  0000 C CNN
+F 1 "TEST_1P" H 9850 1400 50  0000 C CNN
+F 2 "" H 10050 1200 50  0000 C CNN
+F 3 "" H 10050 1200 50  0000 C CNN
+	1    9850 1200
+	1    0    0    -1
+$EndComp
 $EndSCHEMATC
