File: Sch/adc/RF_in.sch (KiCad schematic (older format))
At the start: 72 parts, among them CN1 SMA, CN2 SMA, J3 JP2, J4 JP2, J5 JP2, J6 JP2, U1 LTC2292, U2 BGA2818, U3 TLV702, U4 BGA2818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

Commit message: Adding parts
Parts:
- C12, C22, C24, C25, C37, C38, C39: footprint (none) -> Capacitors_SMD:C_0603
- C23: value 147p -> 150pF; footprint (none) -> Capacitors_SMD:C_0603
- C29, C30, C31, C32, C33, C34, C35, C36, C40: footprint (none) -> Capacitors_SMD:C_0402
- C6: footprint Capacitors_SMD:C_0603 -> Capacitors_SMD:C_0402
- C9: value 10nF -> 0.1uF
- J3, J4, J5, J6: footprint (none) -> Pin_Headers:Pin_Header_Straight_2x02_Pitch2.54mm
Changed lines of the file:
@@
 F 0 "C25" H 2475 1000 50  0000 L CNN
 F 1 "22nF" H 2475 800 50  0000 L CNN
-F 2 "" H 2488 750 50  0001 C CNN
+F 2 "Capacitors_SMD:C_0603" H 2488 750 50  0001 C CNN
 F 3 "" H 2450 900 50  0000 C CNN
 	1    2450 900
@@
 F 0 "C22" H 1475 1700 50  0000 L CNN
 F 1 "18p" H 1475 1500 50  0000 L CNN
-F 2 "" H 1488 1450 50  0001 C CNN
+F 2 "Capacitors_SMD:C_0603" H 1488 1450 50  0001 C CNN
 F 3 "" H 1450 1600 50  0000 C CNN
 	1    1450 1600
@@
 F 0 "C24" H 2325 1700 50  0000 L CNN
 F 1 "18p" H 2325 1500 50  0000 L CNN
-F 2 "" H 2338 1450 50  0001 C CNN
+F 2 "Capacitors_SMD:C_0603" H 2338 1450 50  0001 C CNN
 F 3 "" H 2300 1600 50  0000 C CNN
 	1    2300 1600
@@
 P 1850 2150
 F 0 "C23" H 1875 2250 50  0000 L CNN
-F 1 "147p" H 1875 2050 50  0000 L CNN
-F 2 "" H 1888 2000 50  0001 C CNN
+F 1 "150pF" H 1875 2050 50  0000 L CNN
+F 2 "Capacitors_SMD:C_0603" H 1888 2000 50  0001 C CNN
 F 3 "" H 1850 2150 50  0000 C CNN
 	1    1850 2150
@@
 F 0 "C29" H 9475 2300 50  0000 L CNN
 F 1 "0.1u" H 9475 2100 50  0000 L CNN
-F 2 "" H 9488 2050 50  0001 C CNN
+F 2 "Capacitors_SMD:C_0402" H 9488 2050 50  0001 C CNN
 F 3 "" H 9450 2200 50  0000 C CNN
 	1    9450 2200
@@
 F 0 "C31" H 9725 2300 50  0000 L CNN
 F 1 "2.2u" H 9725 2100 50  0000 L CNN
-F 2 "" H 9738 2050 50  0001 C CNN
+F 2 "Capacitors_SMD:C_0402" H 9738 2050 50  0001 C CNN
 F 3 "" H 9700 2200 50  0000 C CNN
 	1    9700 2200
@@
 F 0 "C33" H 10125 2150 50  0000 L CNN
 F 1 "1u" H 10125 1950 50  0000 L CNN
-F 2 "" H 10138 1900 50  0001 C CNN
+F 2 "Capacitors_SMD:C_0402" H 10138 1900 50  0001 C CNN
 F 3 "" H 10100 2050 50  0000 C CNN
 	1    10100 2050
@@
 F 0 "C34" H 10125 2450 50  0000 L CNN
 F 1 "1u" H 10125 2250 50  0000 L CNN
-F 2 "" H 10138 2200 50  0001 C CNN
+F 2 "Capacitors_SMD:C_0402" H 10138 2200 50  0001 C CNN
 F 3 "" H 10100 2350 50  0000 C CNN
 	1    10100 2350
@@
 F 0 "C30" H 9475 3000 50  0000 L CNN
 F 1 "0.1u" H 9475 2800 50  0000 L CNN
-F 2 "" H 9488 2750 50  0001 C CNN
+F 2 "Capacitors_SMD:C_0402" H 9488 2750 50  0001 C CNN
 F 3 "" H 9450 2900 50  0000 C CNN
 	1    9450 2900
@@
 F 0 "C32" H 9725 3000 50  0000 L CNN
 F 1 "2.2u" H 9725 2800 50  0000 L CNN
-F 2 "" H 9738 2750 50  0001 C CNN
+F 2 "Capacitors_SMD:C_0402" H 9738 2750 50  0001 C CNN
 F 3 "" H 9700 2900 50  0000 C CNN
 	1    9700 2900
@@
 F 0 "C35" H 10125 2850 50  0000 L CNN
 F 1 "1u" H 10125 2650 50  0000 L CNN
-F 2 "" H 10138 2600 50  0001 C CNN
+F 2 "Capacitors_SMD:C_0402" H 10138 2600 50  0001 C CNN
 F 3 "" H 10100 2750 50  0000 C CNN
 	1    10100 2750
@@
 F 0 "C36" H 10125 3150 50  0000 L CNN
 F 1 "1u" H 10125 2950 50  0000 L CNN
-F 2 "" H 10138 2900 50  0001 C CNN
+F 2 "Capacitors_SMD:C_0402" H 10138 2900 50  0001 C CNN
 F 3 "" H 10100 3050 50  0000 C CNN
 	1    10100 3050
@@
 F 0 "C39" H 7175 1900 50  0000 L CNN
 F 1 "12p" H 7175 1700 50  0000 L CNN
-F 2 "" H 7188 1650 50  0001 C CNN
+F 2 "Capacitors_SMD:C_0603" H 7188 1650 50  0001 C CNN
 F 3 "" H 7150 1800 50  0000 C CNN
 	1    7150 1800
@@
 F 0 "C38" H 6625 2500 50  0000 L CNN
 F 1 "0.1u" H 6625 2300 50  0000 L CNN
-F 2 "" H 6638 2250 50  0001 C CNN
+F 2 "Capacitors_SMD:C_0603" H 6638 2250 50  0001 C CNN
 F 3 "" H 6600 2400 50  0000 C CNN
 	1    6600 2400
@@
 F 0 "C40" H 9375 1350 50  0000 L CNN
 F 1 "2.2u" H 9375 1150 50  0000 L CNN
-F 2 "" H 9388 1100 50  0001 C CNN
+F 2 "Capacitors_SMD:C_0402" H 9388 1100 50  0001 C CNN
 F 3 "" H 9350 1250 50  0000 C CNN
 	1    9350 1250
@@
 F 0 "C37" H 4475 2250 50  0000 L CNN
 F 1 "0.1u" H 4475 2050 50  0000 L CNN
-F 2 "" H 4488 2000 50  0001 C CNN
+F 2 "Capacitors_SMD:C_0603" H 4488 2000 50  0001 C CNN
 F 3 "" H 4450 2150 50  0000 C CNN
 	1    4450 2150
@@
 F 0 "J4" H 7200 550 60  0000 C CNN
 F 1 "JP2" H 7200 1000 60  0000 C CNN
-F 2 "" H 7150 900 60  0001 C CNN
+F 2 "Pin_Headers:Pin_Header_Straight_2x02_Pitch2.54mm" H 7150 900 60  0001 C CNN
 F 3 "" H 7150 900 60  0001 C CNN
 	1    7200 800
@@
 F 0 "C6" H 9375 4300 50  0000 L CNN
 F 1 "2.2u" H 9375 4100 50  0000 L CNN
-F 2 "Capacitors_SMD:C_0603" H 9388 4050 50  0001 C CNN
+F 2 "Capacitors_SMD:C_0402" H 9388 4050 50  0001 C CNN
 F 3 "" H 9350 4200 50  0000 C CNN
 	1    9350 4200
@@
 F 0 "J3" H 9300 5050 60  0000 C CNN
 F 1 "JP2" H 9300 5500 60  0000 C CNN
-F 2 "" H 9250 5400 60  0001 C CNN
+F 2 "Pin_Headers:Pin_Header_Straight_2x02_Pitch2.54mm" H 9250 5400 60  0001 C CNN
 F 3 "" H 9250 5400 60  0001 C CNN
 	1    9300 5300
@@
 F 0 "C12" H 5525 2850 50  0000 L CNN
 F 1 "22nF" H 5525 2650 50  0000 L CNN
-F 2 "" H 5538 2600 50  0001 C CNN
+F 2 "Capacitors_SMD:C_0603" H 5538 2600 50  0001 C CNN
 F 3 "" H 5500 2750 50  0000 C CNN
 	1    5500 2750
@@
 P 4700 3200
 F 0 "C9" H 4725 3300 50  0000 L CNN
-F 1 "10nF" H 4725 3100 50  0000 L CNN
+F 1 "0.1uF" H 4725 3100 50  0000 L CNN
 F 2 "Capacitors_SMD:C_0603" H 4738 3050 50  0001 C CNN
 F 3 "" H 4700 3200 50  0000 C CNN
@@
 F 0 "J5" H 4450 3750 60  0000 C CNN
 F 1 "JP2" H 4450 4200 60  0000 C CNN
-F 2 "" H 4400 4100 60  0001 C CNN
+F 2 "Pin_Headers:Pin_Header_Straight_2x02_Pitch2.54mm" H 4400 4100 60  0001 C CNN
 F 3 "" H 4400 4100 60  0001 C CNN
 	1    4450 4000
@@
 F 0 "J6" H 3200 5600 60  0000 C CNN
 F 1 "JP2" H 3200 6050 60  0000 C CNN
-F 2 "" H 3150 5950 60  0001 C CNN
+F 2 "Pin_Headers:Pin_Header_Straight_2x02_Pitch2.54mm" H 3150 5950 60  0001 C CNN
 F 3 "" H 3150 5950 60  0001 C CNN
 	1    3200 5850
