File: Sch/adc/RF_in.sch (KiCad schematic (older format))
At the start: 67 parts, among them CN1 SMA, CN2 SMA, J3 JP2, J4 JP2, T1 ETC1-1-13, U1 LTC2292, U2 LP5907_SOT-23, U3 LP5907_SOT-23, U4 NC7SVU04-SC70, U5 NC7SVU04-SC70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

Commit message: ADC PCB layout in progress
Parts:
- C25: footprint adc_lib:C0603 -> adc_lib:C0402
- R14: footprint adc_lib:R0603 -> adc_lib:R0402
Changed lines of the file:
@@
 $EndComp
 $Comp
-L GND #PWR019
+L GND #PWR018
 U 1 1 58A44759
 P 4950 7300
-F 0 "#PWR019" H 4950 7050 50  0001 C CNN
+F 0 "#PWR018" H 4950 7050 50  0001 C CNN
 F 1 "GND" H 4950 7150 50  0000 C CNN
 F 2 "" H 4950 7300 50  0000 C CNN
@@
 $EndComp
 $Comp
-L GND #PWR020
+L GND #PWR019
 U 1 1 58A3A665
 P 10600 2050
-F 0 "#PWR020" H 10600 1800 50  0001 C CNN
+F 0 "#PWR019" H 10600 1800 50  0001 C CNN
 F 1 "GND" H 10600 1900 50  0000 C CNN
 F 2 "" H 10600 2050 50  0000 C CNN
@@
 $EndComp
 $Comp
-L GND #PWR021
+L GND #PWR020
 U 1 1 58A3A6A7
 P 10600 2350
-F 0 "#PWR021" H 10600 2100 50  0001 C CNN
+F 0 "#PWR020" H 10600 2100 50  0001 C CNN
 F 1 "GND" H 10600 2200 50  0000 C CNN
 F 2 "" H 10600 2350 50  0000 C CNN
@@
 $EndComp
 $Comp
-L GND #PWR022
+L GND #PWR021
 U 1 1 58A3B003
 P 10600 2750
-F 0 "#PWR022" H 10600 2500 50  0001 C CNN
+F 0 "#PWR021" H 10600 2500 50  0001 C CNN
 F 1 "GND" H 10600 2600 50  0000 C CNN
 F 2 "" H 10600 2750 50  0000 C CNN
@@
 $EndComp
 $Comp
-L GND #PWR023
+L GND #PWR022
 U 1 1 58A3B009
 P 10600 3050
-F 0 "#PWR023" H 10600 2800 50  0001 C CNN
+F 0 "#PWR022" H 10600 2800 50  0001 C CNN
 F 1 "GND" H 10600 2900 50  0000 C CNN
 F 2 "" H 10600 3050 50  0000 C CNN
@@
 $EndComp
 $Comp
-L GND #PWR024
+L GND #PWR023
 U 1 1 58A3D81B
 P 9500 1400
-F 0 "#PWR024" H 9500 1150 50  0001 C CNN
+F 0 "#PWR023" H 9500 1150 50  0001 C CNN
 F 1 "GND" H 9500 1250 50  0000 C CNN
 F 2 "" H 9500 1400 50  0000 C CNN
@@
 VCMA
 $Comp
-L GND #PWR025
+L GND #PWR024
 U 1 1 58A5EF6D
 P 2850 7000
-F 0 "#PWR025" H 2850 6750 50  0001 C CNN
+F 0 "#PWR024" H 2850 6750 50  0001 C CNN
 F 1 "GND" H 2850 6850 50  0000 C CNN
 F 2 "" H 2850 7000 50  0000 C CNN
@@
 $EndComp
 $Comp
-L GND #PWR026
+L GND #PWR025
 U 1 1 58A6B351
 P 7850 1200
-F 0 "#PWR026" H 7850 950 50  0001 C CNN
+F 0 "#PWR025" H 7850 950 50  0001 C CNN
 F 1 "GND" H 7850 1050 50  0000 C CNN
 F 2 "" H 7850 1200 50  0000 C CNN
@@
 VCMA
 $Comp
-L GND #PWR027
+L GND #PWR026
 U 1 1 58A6C57D
 P 9500 4350
-F 0 "#PWR027" H 9500 4100 50  0001 C CNN
+F 0 "#PWR026" H 9500 4100 50  0001 C CNN
 F 1 "GND" H 9500 4200 50  0000 C CNN
 F 2 "" H 9500 4350 50  0000 C CNN
@@
 $EndComp
 $Comp
-L GND #PWR028
+L GND #PWR027
 U 1 1 58A6CD2B
 P 9950 5700
-F 0 "#PWR028" H 9950 5450 50  0001 C CNN
+F 0 "#PWR027" H 9950 5450 50  0001 C CNN
 F 1 "GND" H 9950 5550 50  0000 C CNN
 F 2 "" H 9950 5700 50  0000 C CNN
@@
 ADC_CLK
 $Comp
-L GND #PWR029
+L GND #PWR028
 U 1 1 58A70E23
 P 4200 7000
-F 0 "#PWR029" H 4200 6750 50  0001 C CNN
+F 0 "#PWR028" H 4200 6750 50  0001 C CNN
 F 1 "GND" H 4200 6850 50  0000 C CNN
 F 2 "" H 4200 7000 50  0000 C CNN
@@
 $EndComp
 $Comp
-L GND #PWR030
+L GND #PWR029
 U 1 1 58A70EA4
 P 4400 7000
-F 0 "#PWR030" H 4400 6750 50  0001 C CNN
+F 0 "#PWR029" H 4400 6750 50  0001 C CNN
 F 1 "GND" H 4400 6850 50  0000 C CNN
 F 2 "" H 4400 7000 50  0000 C CNN
@@
 $EndComp
 $Comp
-L GND #PWR031
+L GND #PWR030
 U 1 1 58A70F2D
 P 4600 7000
-F 0 "#PWR031" H 4600 6750 50  0001 C CNN
+F 0 "#PWR030" H 4600 6750 50  0001 C CNN
 F 1 "GND" H 4600 6850 50  0000 C CNN
 F 2 "" H 4600 7000 50  0000 C CNN
@@
 $EndComp
 $Comp
-L GND #PWR032
+L GND #PWR031
 U 1 1 58A70FB2
 P 4800 7000
-F 0 "#PWR032" H 4800 6750 50  0001 C CNN
+F 0 "#PWR031" H 4800 6750 50  0001 C CNN
 F 1 "GND" H 4800 6850 50  0000 C CNN
 F 2 "" H 4800 7000 50  0000 C CNN
@@
 $EndComp
 $Comp
-L GND #PWR033
+L GND #PWR032
 U 1 1 58A72283
 P 5400 7500
-F 0 "#PWR033" H 5400 7250 50  0001 C CNN
+F 0 "#PWR032" H 5400 7250 50  0001 C CNN
 F 1 "GND" H 5400 7350 50  0000 C CNN
 F 2 "" H 5400 7500 50  0000 C CNN
@@
 $EndComp
 $Comp
-L GND #PWR034
+L GND #PWR033
 U 1 1 58A72318
 P 5600 7500
-F 0 "#PWR034" H 5600 7250 50  0001 C CNN
+F 0 "#PWR033" H 5600 7250 50  0001 C CNN
 F 1 "GND" H 5600 7350 50  0000 C CNN
 F 2 "" H 5600 7500 50  0000 C CNN
@@
 VCMB
 $Comp
-L GND #PWR035
+L GND #PWR034
 U 1 1 58A75DF8
 P 7150 4000
-F 0 "#PWR035" H 7150 3750 50  0001 C CNN
+F 0 "#PWR034" H 7150 3750 50  0001 C CNN
 F 1 "GND" H 7150 3850 50  0000 C CNN
 F 2 "" H 7150 4000 50  0000 C CNN
@@
 VDD: 2Vp-p,\nVCM: 1Vp-p
 $Comp
-L GND #PWR036
+L GND #PWR035
 U 1 1 58A8E85E
 P 5650 3350
-F 0 "#PWR036" H 5650 3100 50  0001 C CNN
+F 0 "#PWR035" H 5650 3100 50  0001 C CNN
 F 1 "GND" H 5650 3200 50  0000 C CNN
 F 2 "" H 5650 3350 50  0000 C CNN
@@
 F 0 "R14" V 4830 4500 50  0000 C CNN
 F 1 "0" V 4750 4500 50  0000 C CNN
-F 2 "adc_lib:R0603" V 4680 4500 50  0001 C CNN
+F 2 "adc_lib:R0402" V 4680 4500 50  0001 C CNN
 F 3 "" H 4750 4500 50  0000 C CNN
 	1    4750 4500
@@
 $EndComp
 $Comp
-L GND #PWR037
+L GND #PWR036
 U 1 1 595093B3
 P 900 4850
-F 0 "#PWR037" H 900 4600 50  0001 C CNN
+F 0 "#PWR036" H 900 4600 50  0001 C CNN
 F 1 "GND" H 900 4700 50  0000 C CNN
 F 2 "" H 900 4850 50  0000 C CNN
@@
 NoConn ~ 2350 4650
 $Comp
-L GND #PWR038
+L GND #PWR037
 U 1 1 5955200C
 P 2350 4950
-F 0 "#PWR038" H 2350 4700 50  0001 C CNN
+F 0 "#PWR037" H 2350 4700 50  0001 C CNN
 F 1 "GND" H 2350 4800 50  0000 C CNN
 F 2 "" H 2350 4950 50  0000 C CNN
@@
 $EndComp
 $Comp
-L GND #PWR039
+L GND #PWR038
 U 1 1 59553EA1
 P 3350 4250
-F 0 "#PWR039" H 3350 4000 50  0001 C CNN
+F 0 "#PWR038" H 3350 4000 50  0001 C CNN
 F 1 "GND" H 3350 4100 50  0000 C CNN
 F 2 "" H 3350 4250 50  0000 C CNN
@@
 $EndComp
 $Comp
-L GND #PWR040
+L GND #PWR039
 U 1 1 59555903
 P 3600 5050
-F 0 "#PWR040" H 3600 4800 50  0001 C CNN
+F 0 "#PWR039" H 3600 4800 50  0001 C CNN
 F 1 "GND" H 3600 4900 50  0000 C CNN
 F 2 "" H 3600 5050 50  0000 C CNN
@@
 $EndComp
 $Comp
-L GND #PWR041
+L GND #PWR040
 U 1 1 595586F8
 P 4150 4250
-F 0 "#PWR041" H 4150 4000 50  0001 C CNN
+F 0 "#PWR040" H 4150 4000 50  0001 C CNN
 F 1 "GND" H 4150 4100 50  0000 C CNN
 F 2 "" H 4150 4250 50  0000 C CNN
@@
 $EndComp
 $Comp
-L GND #PWR042
+L GND #PWR041
 U 1 1 59559CFF
 P 2850 4250
-F 0 "#PWR042" H 2850 4000 50  0001 C CNN
+F 0 "#PWR041" H 2850 4000 50  0001 C CNN
 F 1 "GND" H 2850 4100 50  0000 C CNN
 F 2 "" H 2850 4250 50  0000 C CNN
@@
 $EndComp
 $Comp
-L GND #PWR043
+L GND #PWR042
 U 1 1 595645F8
 P 5950 2150
-F 0 "#PWR043" H 5950 1900 50  0001 C CNN
+F 0 "#PWR042" H 5950 1900 50  0001 C CNN
 F 1 "GND" H 5950 2000 50  0000 C CNN
 F 2 "" H 5950 2150 50  0000 C CNN
@@
 F 0 "C25" H 7225 1850 50  0000 L CNN
 F 1 "0.1u" H 7225 1650 50  0000 L CNN
-F 2 "adc_lib:C0603" H 7238 1600 50  0001 C CNN
+F 2 "adc_lib:C0402" H 7238 1600 50  0001 C CNN
 F 3 "" H 7200 1750 50  0000 C CNN
 	1    7200 1750
@@
 $EndComp
 $Comp
-L GND #PWR044
+L GND #PWR043
 U 1 1 59565C5A
 P 7350 1750
-F 0 "#PWR044" H 7350 1500 50  0001 C CNN
+F 0 "#PWR043" H 7350 1500 50  0001 C CNN
 F 1 "GND" H 7350 1600 50  0000 C CNN
 F 2 "" H 7350 1750 50  0000 C CNN
@@
 	6700 1300 6450 1300
 $Comp
-L GND #PWR045
+L GND #PWR044
 U 1 1 5956B4E5
 P 4700 1800
-F 0 "#PWR045" H 4700 1550 50  0001 C CNN
+F 0 "#PWR044" H 4700 1550 50  0001 C CNN
 F 1 "GND" H 4700 1650 50  0000 C CNN
 F 2 "" H 4700 1800 50  0000 C CNN
@@
 $EndComp
 $Comp
-L +3V3 #PWR046
+L +3V3 #PWR045
 U 1 1 5956828F
 P 4250 5500
-F 0 "#PWR046" H 4250 5350 50  0001 C CNN
+F 0 "#PWR045" H 4250 5350 50  0001 C CNN
 F 1 "+3V3" H 4250 5640 50  0000 C CNN
 F 2 "" H 4250 5500 50  0000 C CNN
@@
 	3050 7000 3050 6900
 $Comp
-L GND #PWR047
+L GND #PWR046
 U 1 1 5956A6B3
 P 2850 3400
-F 0 "#PWR047" H 2850 3150 50  0001 C CNN
+F 0 "#PWR046" H 2850 3150 50  0001 C CNN
 F 1 "GND" H 2850 3250 50  0000 C CNN
 F 2 "" H 2850 3400 50  0000 C CNN
@@
 $EndComp
 $Comp
-L +5V #PWR048
+L +5V #PWR047
 U 1 1 598044DD
 P 850 700
-F 0 "#PWR048" H 850 550 50  0001 C CNN
+F 0 "#PWR047" H 850 550 50  0001 C CNN
 F 1 "+5V" H 850 840 50  0000 C CNN
 F 2 "" H 850 700 50  0000 C CNN
@@
 $EndComp
 $Comp
-L GND #PWR049
+L GND #PWR048
 U 1 1 598046E8
 P 1200 1450
-F 0 "#PWR049" H 1200 1200 50  0001 C CNN
+F 0 "#PWR048" H 1200 1200 50  0001 C CNN
 F 1 "GND" H 1200 1300 50  0000 C CNN
 F 2 "" H 1200 1450 50  0000 C CNN
@@
 $EndComp
 $Comp
-L GND #PWR050
+L GND #PWR049
 U 1 1 59804AC2
 P 2050 1450
-F 0 "#PWR050" H 2050 1200 50  0001 C CNN
+F 0 "#PWR049" H 2050 1200 50  0001 C CNN
 F 1 "GND" H 2050 1300 50  0000 C CNN
 F 2 "" H 2050 1450 50  0000 C CNN

Commit message: Add GND and more layout
Parts:
- removed C19: 4.7u 6V, adc_lib:C0603, symbol C
- CN1, CN2: footprint adc_lib:SMA_RightAngle -> adc_lib:SMA_Edge
Other:
- note removed: "Is this required?"
Changed lines of the file:
@@
 F 0 "CN1" H 5100 1350 60  0000 C CNN
 F 1 "SMA" H 5100 1950 60  0000 C CNN
-F 2 "adc_lib:SMA_RightAngle" H 5000 1650 60  0001 C CNN
+F 2 "adc_lib:SMA_Edge" H 5000 1650 60  0001 C CNN
 F 3 "" H 5000 1650 60  0001 C CNN
 	1    5100 1650
@@
 F 0 "CN2" H 6050 2900 60  0000 C CNN
 F 1 "SMA" H 6050 3500 60  0000 C CNN
-F 2 "adc_lib:SMA_RightAngle" H 5950 3200 60  0001 C CNN
+F 2 "adc_lib:SMA_Edge" H 5950 3200 60  0001 C CNN
 F 3 "" H 5950 3200 60  0001 C CNN
 	1    6050 3200
@@
 	1    0    0    -1
 $EndComp
-$Comp
-L C C19
-U 1 1 59559CF9
-P 2850 4100
-F 0 "C19" H 2875 4200 50  0000 L CNN
-F 1 "4.7u 6V" H 2875 4000 50  0000 L CNN
-F 2 "adc_lib:C0603" H 2888 3950 50  0001 C CNN
-F 3 "" H 2850 4100 50  0000 C CNN
-	1    2850 4100
-	1    0    0    -1
-$EndComp
-$Comp
-L GND #PWR041
-U 1 1 59559CFF
-P 2850 4250
-F 0 "#PWR041" H 2850 4000 50  0001 C CNN
-F 1 "GND" H 2850 4100 50  0000 C CNN
-F 2 "" H 2850 4250 50  0000 C CNN
-F 3 "" H 2850 4250 50  0000 C CNN
-	1    2850 4250
-	1    0    0    -1
-$EndComp
 NoConn ~ 3600 4750
 $Comp
@@
 $EndComp
 $Comp
-L GND #PWR042
+L GND #PWR041
 U 1 1 595645F8
 P 5950 2150
-F 0 "#PWR042" H 5950 1900 50  0001 C CNN
+F 0 "#PWR041" H 5950 1900 50  0001 C CNN
 F 1 "GND" H 5950 2000 50  0000 C CNN
 F 2 "" H 5950 2150 50  0000 C CNN
@@
 $EndComp
 $Comp
-L GND #PWR043
+L GND #PWR042
 U 1 1 59565C5A
 P 7350 1750
-F 0 "#PWR043" H 7350 1500 50  0001 C CNN
+F 0 "#PWR042" H 7350 1500 50  0001 C CNN
 F 1 "GND" H 7350 1600 50  0000 C CNN
 F 2 "" H 7350 1750 50  0000 C CNN
@@
 	4400 3950 4400 4750
 Connection ~ 4150 3950
-Connection ~ 2850 3950
 Wire Wire Line
 	4900 4500 5350 4500
@@
 	6700 1300 6450 1300
 $Comp
-L GND #PWR044
+L GND #PWR043
 U 1 1 5956B4E5
 P 4700 1800
-F 0 "#PWR044" H 4700 1550 50  0001 C CNN
+F 0 "#PWR043" H 4700 1550 50  0001 C CNN
 F 1 "GND" H 4700 1650 50  0000 C CNN
 F 2 "" H 4700 1800 50  0000 C CNN
@@
 $EndComp
 $Comp
-L +3V3 #PWR045
+L +3V3 #PWR044
 U 1 1 5956828F
 P 4250 5500
-F 0 "#PWR045" H 4250 5350 50  0001 C CNN
+F 0 "#PWR044" H 4250 5350 50  0001 C CNN
 F 1 "+3V3" H 4250 5640 50  0000 C CNN
 F 2 "" H 4250 5500 50  0000 C CNN
@@
 	3050 7000 3050 6900
 $Comp
-L GND #PWR046
+L GND #PWR045
 U 1 1 5956A6B3
 P 2850 3400
-F 0 "#PWR046" H 2850 3150 50  0001 C CNN
+F 0 "#PWR045" H 2850 3150 50  0001 C CNN
 F 1 "GND" H 2850 3250 50  0000 C CNN
 F 2 "" H 2850 3400 50  0000 C CNN
@@
 	1950 3750 1950 3950
 Connection ~ 1950 3950
-Text Notes 2350 3900 0    60   ~ 0
-Is this required?
 Text Label 2850 800  0    60   ~ 0
 VCC5
@@
 $EndComp
 $Comp
-L +5V #PWR047
+L +5V #PWR046
 U 1 1 598044DD
 P 850 700
-F 0 "#PWR047" H 850 550 50  0001 C CNN
+F 0 "#PWR046" H 850 550 50  0001 C CNN
 F 1 "+5V" H 850 840 50  0000 C CNN
 F 2 "" H 850 700 50  0000 C CNN
@@
 $EndComp
 $Comp
-L GND #PWR048
+L GND #PWR047
 U 1 1 598046E8
 P 1200 1450
-F 0 "#PWR048" H 1200 1200 50  0001 C CNN
+F 0 "#PWR047" H 1200 1200 50  0001 C CNN
 F 1 "GND" H 1200 1300 50  0000 C CNN
 F 2 "" H 1200 1450 50  0000 C CNN
@@
 $EndComp
 $Comp
-L GND #PWR049
+L GND #PWR048
 U 1 1 59804AC2
 P 2050 1450
-F 0 "#PWR049" H 2050 1200 50  0001 C CNN
+F 0 "#PWR048" H 2050 1200 50  0001 C CNN
 F 1 "GND" H 2050 1300 50  0000 C CNN
 F 2 "" H 2050 1450 50  0000 C CNN

Commit message: Improve layout
Connections:
- net labels added: VDD3_2
Changed lines of the file:
@@
 $EndComp
 Wire Wire Line
-	1200 3950 4400 3950
+	1200 3950 4650 3950
+Text GLabel 4650 3950 2    60   Output ~ 0
+VDD3_2
+Connection ~ 4400 3950
 $EndSCHEMATC
