File: Sch/fm_bpf/fm_bpf.sch (KiCad schematic (older format))
At the start: 27 parts

Commit message: Start BOM for BPF
Parts:
- added R2: 10k, symbol R
- gave numbers to parts that had none: 27
Connections:
- net +5V: now also U1.1 (IN), R2.1
- net at U1.3 (EN): now also R2.2
Other:
- note added: "410mOhm"
- note added: "LNA Max 66mA"
Changed lines of the file:
@@
 LIBS:valves
 LIBS:zturn_adc
-LIBS:CYUSB3014
 LIBS:fm_bpf-cache
 EELAYER 25 0
@@
 $EndDescr
 $Comp
-L SMA CN?
+L SMA CN1
 U 1 1 59784837
 P 2150 2800
-F 0 "CN?" H 2150 2500 60  0000 C CNN
+F 0 "CN1" H 2150 2500 60  0000 C CNN
 F 1 "SMA" H 2150 3100 60  0000 C CNN
 F 2 "" H 2050 2800 60  0001 C CNN
@@
 $EndComp
 $Comp
-L SMA CN?
+L SMA CN2
 U 1 1 59784880
 P 9400 3000
-F 0 "CN?" H 9400 2700 60  0000 C CNN
+F 0 "CN2" H 9400 2700 60  0000 C CNN
 F 1 "SMA" H 9400 3300 60  0000 C CNN
 F 2 "" H 9300 3000 60  0001 C CNN
@@
 $EndComp
 $Comp
-L JP2 J?
+L JP2 J1
 U 1 1 597848E9
 P 1600 5000
-F 0 "J?" H 1600 4750 60  0000 C CNN
+F 0 "J1" H 1600 4750 60  0000 C CNN
 F 1 "JP2" H 1600 5200 60  0000 C CNN
 F 2 "" H 1550 5100 60  0001 C CNN
@@
 $EndComp
 $Comp
-L +3V3 #PWR?
+L +3V3 #PWR01
 U 1 1 59784946
 P 1050 4850
-F 0 "#PWR?" H 1050 4700 50  0001 C CNN
+F 0 "#PWR01" H 1050 4700 50  0001 C CNN
 F 1 "+3V3" H 1050 4990 50  0000 C CNN
 F 2 "" H 1050 4850 50  0000 C CNN
@@
 $EndComp
 $Comp
-L +5V #PWR?
+L +5V #PWR02
 U 1 1 59784960
 P 2100 4850
-F 0 "#PWR?" H 2100 4700 50  0001 C CNN
+F 0 "#PWR02" H 2100 4700 50  0001 C CNN
 F 1 "+5V" H 2100 4990 50  0000 C CNN
 F 2 "" H 2100 4850 50  0000 C CNN
@@
 $EndComp
 $Comp
-L GND #PWR?
+L GND #PWR03
 U 1 1 597849CB
 P 1050 5350
-F 0 "#PWR?" H 1050 5100 50  0001 C CNN
+F 0 "#PWR03" H 1050 5100 50  0001 C CNN
 F 1 "GND" H 1050 5200 50  0000 C CNN
 F 2 "" H 1050 5350 50  0000 C CNN
@@
 $EndComp
 $Comp
-L LP5907_SOT-23 U?
+L LP5907_SOT-23 U1
 U 1 1 59784B61
 P 2900 1600
-F 0 "U?" H 2900 1300 60  0000 C CNN
+F 0 "U1" H 2900 1300 60  0000 C CNN
 F 1 "LP5907_SOT-23" H 2900 1900 60  0000 C CNN
 F 2 "" H 2900 1300 60  0001 C CNN
@@
 $EndComp
 $Comp
-L GND #PWR?
+L GND #PWR04
 U 1 1 59784C9E
 P 1550 3200
-F 0 "#PWR?" H 1550 2950 50  0001 C CNN
+F 0 "#PWR04" H 1550 2950 50  0001 C CNN
 F 1 "GND" H 1550 3050 50  0000 C CNN
 F 2 "" H 1550 3200 50  0000 C CNN
@@
 250mA Vo=3.8V (LP5907QMFX-3.8Q1)
 $Comp
-L C C?
+L C C1
 U 1 1 5979F339
 P 2050 1850
-F 0 "C?" H 2075 1950 50  0000 L CNN
+F 0 "C1" H 2075 1950 50  0000 L CNN
 F 1 "1u" H 2075 1750 50  0000 L CNN
 F 2 "" H 2088 1700 50  0000 C CNN
@@
 $EndComp
 $Comp
-L C C?
+L C C4
 U 1 1 5979F374
 P 3600 1850
-F 0 "C?" H 3625 1950 50  0000 L CNN
+F 0 "C4" H 3625 1950 50  0000 L CNN
 F 1 "1u" H 3625 1750 50  0000 L CNN
 F 2 "" H 3638 1700 50  0000 C CNN
@@
 $EndComp
 $Comp
-L GND #PWR?
+L GND #PWR05
 U 1 1 5979F3B6
 P 2400 2100
-F 0 "#PWR?" H 2400 1850 50  0001 C CNN
+F 0 "#PWR05" H 2400 1850 50  0001 C CNN
 F 1 "GND" H 2400 1950 50  0000 C CNN
 F 2 "" H 2400 2100 50  0000 C CNN
@@
 NoConn ~ 3350 1700
 $Comp
-L +5V #PWR?
+L +5V #PWR06
 U 1 1 5979F65E
 P 2050 1350
-F 0 "#PWR?" H 2050 1200 50  0001 C CNN
+F 0 "#PWR06" H 2050 1200 50  0001 C CNN
 F 1 "+5V" H 2050 1490 50  0000 C CNN
 F 2 "" H 2050 1350 50  0000 C CNN
@@
 $EndComp
 $Comp
-L R R?
+L R R1
 U 1 1 5979F787
 P 4550 1500
-F 0 "R?" V 4630 1500 50  0000 C CNN
+F 0 "R1" V 4630 1500 50  0000 C CNN
 F 1 "680" V 4550 1500 50  0000 C CNN
 F 2 "" V 4480 1500 50  0000 C CNN
@@
 $EndComp
 $Comp
-L L L?
+L L L3
 U 1 1 5979F7CE
 P 4550 1750
-F 0 "L?" V 4500 1750 50  0000 C CNN
+F 0 "L3" V 4500 1750 50  0000 C CNN
 F 1 "8.2u" V 4625 1750 50  0000 C CNN
 F 2 "" H 4550 1750 50  0000 C CNN
@@
 $EndComp
 $Comp
-L C C?
+L C C6
 U 1 1 5979F81A
 P 4200 1900
-F 0 "C?" H 4225 2000 50  0000 L CNN
+F 0 "C6" H 4225 2000 50  0000 L CNN
 F 1 "0.1u" H 4225 1800 50  0000 L CNN
 F 2 "" H 4238 1750 50  0000 C CNN
@@
 $EndComp
 $Comp
-L GND #PWR?
+L GND #PWR07
 U 1 1 5979F98F
 P 4200 2050
-F 0 "#PWR?" H 4200 1800 50  0001 C CNN
+F 0 "#PWR07" H 4200 1800 50  0001 C CNN
 F 1 "GND" H 4200 1900 50  0000 C CNN
 F 2 "" H 4200 2050 50  0000 C CNN
@@
 $EndComp
 $Comp
-L C C?
+L C C8
 U 1 1 5979FA8B
 P 5200 1900
-F 0 "C?" H 5225 2000 50  0000 L CNN
+F 0 "C8" H 5225 2000 50  0000 L CNN
 F 1 "0.1u" H 5225 1800 50  0000 L CNN
 F 2 "" H 5238 1750 50  0000 C CNN
@@
 $EndComp
 $Comp
-L GND #PWR?
+L GND #PWR08
 U 1 1 5979FA91
 P 5200 2050
-F 0 "#PWR?" H 5200 1800 50  0001 C CNN
+F 0 "#PWR08" H 5200 1800 50  0001 C CNN
 F 1 "GND" H 5200 1900 50  0000 C CNN
 F 2 "" H 5200 2050 50  0000 C CNN
@@
 $EndComp
 $Comp
-L L L?
+L L L4
 U 1 1 5979FAC0
 P 5500 1500
-F 0 "L?" V 5450 1500 50  0000 C CNN
+F 0 "L4" V 5450 1500 50  0000 C CNN
 F 1 "3.3u" V 5575 1500 50  0000 C CNN
 F 2 "" H 5500 1500 50  0000 C CNN
@@
 $EndComp
 $Comp
-L PSA4-5043+ U?
+L PSA4-5043+ U2
 U 1 1 5979FFAD
 P 5300 2900
-F 0 "U?" H 5600 2600 60  0000 C CNN
+F 0 "U2" H 5600 2600 60  0000 C CNN
 F 1 "PSA4-5043+" H 5150 3150 60  0000 C CNN
 F 2 "" H 5150 3150 60  0001 C CNN
@@
 $EndComp
 $Comp
-L GND #PWR?
+L GND #PWR09
 U 1 1 597A0121
 P 4600 3250
-F 0 "#PWR?" H 4600 3000 50  0001 C CNN
+F 0 "#PWR09" H 4600 3000 50  0001 C CNN
 F 1 "GND" H 4600 3100 50  0000 C CNN
 F 2 "" H 4600 3250 50  0000 C CNN
@@
 	5950 3000 6550 3000
 $Comp
-L C C?
+L C C2
 U 1 1 597A03A5
 P 2750 2950
-F 0 "C?" H 2775 3050 50  0000 L CNN
+F 0 "C2" H 2775 3050 50  0000 L CNN
 F 1 "27p" H 2775 2850 50  0000 L CNN
 F 2 "" H 2788 2800 50  0000 C CNN
@@
 $EndComp
 $Comp
-L C C?
+L C C3
 U 1 1 597A0430
 P 3100 2800
-F 0 "C?" H 3125 2900 50  0000 L CNN
+F 0 "C3" H 3125 2900 50  0000 L CNN
 F 1 "12p" H 3125 2700 50  0000 L CNN
 F 2 "" H 3138 2650 50  0000 C CNN
@@
 $EndComp
 $Comp
-L L L?
+L L L1
 U 1 1 597A04AF
 P 3400 2800
-F 0 "L?" V 3350 2800 50  0000 C CNN
+F 0 "L1" V 3350 2800 50  0000 C CNN
 F 1 "330n" V 3475 2800 50  0000 C CNN
 F 2 "" H 3400 2800 50  0000 C CNN
@@
 $EndComp
 $Comp
-L L L?
+L L L2
 U 1 1 597A04F6
 P 3650 2950
-F 0 "L?" V 3600 2950 50  0000 C CNN
+F 0 "L2" V 3600 2950 50  0000 C CNN
 F 1 "27n" V 3725 2950 50  0000 C CNN
 F 2 "" H 3650 2950 50  0000 C CNN
@@
 $EndComp
 $Comp
-L C C?
+L C C5
 U 1 1 597A0623
 P 3950 2950
-F 0 "C?" H 3975 3050 50  0000 L CNN
+F 0 "C5" H 3975 3050 50  0000 L CNN
 F 1 "130p" H 3975 2850 50  0000 L CNN
 F 2 "" H 3988 2800 50  0000 C CNN
@@
 $EndComp
 $Comp
-L GND #PWR?
+L GND #PWR010
 U 1 1 597A07B7
 P 2750 3200
-F 0 "#PWR?" H 2750 2950 50  0001 C CNN
+F 0 "#PWR010" H 2750 2950 50  0001 C CNN
 F 1 "GND" H 2750 3050 50  0000 C CNN
 F 2 "" H 2750 3200 50  0000 C CNN
@@
 Connection ~ 3650 3100
 $Comp
-L C C?
+L C C7
 U 1 1 597A0C19
 P 4350 2800
-F 0 "C?" H 4375 2900 50  0000 L CNN
+F 0 "C7" H 4375 2900 50  0000 L CNN
 F 1 "0.1u" H 4375 2700 50  0000 L CNN
 F 2 "" H 4388 2650 50  0000 C CNN
@@
 	4500 2800 4700 2800
 $Comp
-L C C?
+L C C10
 U 1 1 597A0FE1
 P 6700 3000
-F 0 "C?" H 6725 3100 50  0000 L CNN
+F 0 "C10" H 6725 3100 50  0000 L CNN
 F 1 "5p" H 6725 2900 50  0000 L CNN
 F 2 "" H 6738 2850 50  0000 C CNN
@@
 $EndComp
 $Comp
-L C C?
+L C C9
 U 1 1 597A1122
 P 6700 2700
-F 0 "C?" H 6725 2800 50  0000 L CNN
+F 0 "C9" H 6725 2800 50  0000 L CNN
 F 1 "9p" H 6725 2600 50  0000 L CNN
 F 2 "" H 6738 2550 50  0000 C CNN
@@
 $EndComp
 $Comp
-L L L?
+L L L5
 U 1 1 597A11DE
 P 7000 3000
-F 0 "L?" V 6950 3000 50  0000 C CNN
+F 0 "L5" V 6950 3000 50  0000 C CNN
 F 1 "560n" V 7075 3000 50  0000 C CNN
 F 2 "" H 7000 3000 50  0000 C CNN
@@
 $EndComp
 $Comp
-L L L?
+L L L6
 U 1 1 597A1239
 P 7450 3150
-F 0 "L?" V 7400 3150 50  0000 C CNN
+F 0 "L6" V 7400 3150 50  0000 C CNN
 F 1 "100n" V 7525 3150 50  0000 C CNN
 F 2 "" H 7450 3150 50  0000 C CNN
@@
 $EndComp
 $Comp
-L C C?
+L C C11
 U 1 1 597A12FD
 P 7450 3450
-F 0 "C?" H 7475 3550 50  0000 L CNN
+F 0 "C11" H 7475 3550 50  0000 L CNN
 F 1 "68p" H 7475 3350 50  0000 L CNN
 F 2 "" H 7488 3300 50  0000 C CNN
@@
 $EndComp
 $Comp
-L C C?
+L C C12
 U 1 1 597A1393
 P 7800 3450
-F 0 "C?" H 7825 3550 50  0000 L CNN
+F 0 "C12" H 7825 3550 50  0000 L CNN
 F 1 "82p" H 7825 3350 50  0000 L CNN
 F 2 "" H 7838 3300 50  0000 C CNN
@@
 $EndComp
 $Comp
-L L L?
+L L L7
 U 1 1 597A13FF
 P 8100 3000
-F 0 "L?" V 8050 3000 50  0000 C CNN
+F 0 "L7" V 8050 3000 50  0000 C CNN
 F 1 "560n" V 8175 3000 50  0000 C CNN
 F 2 "" H 8100 3000 50  0000 C CNN
@@
 $EndComp
 $Comp
-L C C?
+L C C13
 U 1 1 597A148D
 P 8400 2750
-F 0 "C?" H 8425 2850 50  0000 L CNN
+F 0 "C13" H 8425 2850 50  0000 L CNN
 F 1 "5p" H 8425 2650 50  0000 L CNN
 F 2 "" H 8438 2600 50  0000 C CNN
@@
 $EndComp
 $Comp
-L C C?
+L C C14
 U 1 1 597A14DE
 P 8400 3000
-F 0 "C?" H 8425 3100 50  0000 L CNN
+F 0 "C14" H 8425 3100 50  0000 L CNN
 F 1 "5p" H 8425 2900 50  0000 L CNN
 F 2 "" H 8438 2850 50  0000 C CNN
@@
 	6400 2700 6400 3000
 $Comp
-L GND #PWR?
+L GND #PWR011
 U 1 1 597A19E1
 P 7450 3750
-F 0 "#PWR?" H 7450 3500 50  0001 C CNN
+F 0 "#PWR011" H 7450 3500 50  0001 C CNN
 F 1 "GND" H 7450 3600 50  0000 C CNN
 F 2 "" H 7450 3750 50  0000 C CNN
@@
 Connection ~ 8700 3000
 $Comp
-L GND #PWR?
+L GND #PWR012
 U 1 1 597A2125
 P 9950 3350
-F 0 "#PWR?" H 9950 3100 50  0001 C CNN
+F 0 "#PWR012" H 9950 3100 50  0001 C CNN
 F 1 "GND" H 9950 3200 50  0000 C CNN
 F 2 "" H 9950 3350 50  0000 C CNN
@@
 Text Notes 3000 2600 0    60   ~ 0
 BPF 72-96MHz
+Text Notes 5200 2600 0    60   ~ 0
+LNA Max 66mA
+$Comp
+L R R2
+U 1 1 597B03B9
+P 2350 1700
+F 0 "R2" V 2430 1700 50  0000 C CNN
+F 1 "10k" V 2350 1700 50  0000 C CNN
+F 2 "" V 2280 1700 50  0000 C CNN
+F 3 "" H 2350 1700 50  0000 C CNN
+	1    2350 1700
+	0    -1   -1   0
+$EndComp
+Wire Wire Line
+	2200 1700 2200 1500
+Connection ~ 2200 1500
+Connection ~ 2050 1500
+$Comp
+L PWR_FLAG #FLG013
+U 1 1 597B088B
+P 2450 4850
+F 0 "#FLG013" H 2450 4945 50  0001 C CNN
+F 1 "PWR_FLAG" H 2450 5030 50  0000 C CNN
+F 2 "" H 2450 4850 50  0000 C CNN
+F 3 "" H 2450 4850 50  0000 C CNN
+	1    2450 4850
+	1    0    0    -1
+$EndComp
+Wire Wire Line
+	2450 4850 2450 4900
+Wire Wire Line
+	2450 4900 2100 4900
+Connection ~ 2100 4900
+Text Notes 4500 2000 0    60   ~ 0
+410mOhm
 $EndSCHEMATC

Commit message: BOM list done
Parts:
- C12: value 82p -> 100p
Other:
- note added: "230mOhm"
Changed lines of the file:
@@
 P 7800 3450
 F 0 "C12" H 7825 3550 50  0000 L CNN
-F 1 "82p" H 7825 3350 50  0000 L CNN
+F 1 "100p" H 7825 3350 50  0000 L CNN
 F 2 "" H 7838 3300 50  0000 C CNN
 F 3 "" H 7800 3450 50  0000 C CNN
@@
 Text Notes 4500 2000 0    60   ~ 0
 410mOhm
+Text Notes 5400 1700 0    60   ~ 0
+230mOhm
 $EndSCHEMATC

Commit message: Start PCB design
Parts:
- removed CN1, CN2: SMA, symbol SMA
- added CN1, CN2: SMA_Edge, adc_lib:SMA_Edge, symbol SMA_Edge
- C1, C10, C11, C12, C13, C14, C2, C3, C4, C5, C6, C7, C8, C9: footprint (none) -> adc_lib:C0603
- J1: footprint (none) -> adc_lib:M20-9980245
- L1, L2, L4, L5, L6, L7: footprint (none) -> adc_lib:L0603
- L3: footprint (none) -> adc_lib:L1008
- R1, R2: footprint (none) -> adc_lib:R0603
- U1: footprint (none) -> adc_lib:LP5907
- U2: footprint (none) -> adc_lib:MMM1362
Connections:
- wire segments 61 -> 57
Changed lines of the file:
@@
 $EndDescr
-$Comp
-L SMA CN1
-U 1 1 59784837
-P 2150 2800
-F 0 "CN1" H 2150 2500 60  0000 C CNN
-F 1 "SMA" H 2150 3100 60  0000 C CNN
-F 2 "" H 2050 2800 60  0001 C CNN
-F 3 "" H 2050 2800 60  0001 C CNN
-	1    2150 2800
-	-1   0    0    1
-$EndComp
-$Comp
-L SMA CN2
-U 1 1 59784880
-P 9400 3000
-F 0 "CN2" H 9400 2700 60  0000 C CNN
-F 1 "SMA" H 9400 3300 60  0000 C CNN
-F 2 "" H 9300 3000 60  0001 C CNN
-F 3 "" H 9300 3000 60  0001 C CNN
-	1    9400 3000
-	1    0    0    -1
-$EndComp
 $Comp
 L JP2 J1
@@
 F 0 "J1" H 1600 4750 60  0000 C CNN
 F 1 "JP2" H 1600 5200 60  0000 C CNN
-F 2 "" H 1550 5100 60  0001 C CNN
+F 2 "adc_lib:M20-9980245" H 1550 5100 60  0001 C CNN
 F 3 "" H 1550 5100 60  0001 C CNN
 	1    1600 5000
@@
 F 0 "U1" H 2900 1300 60  0000 C CNN
 F 1 "LP5907_SOT-23" H 2900 1900 60  0000 C CNN
-F 2 "" H 2900 1300 60  0001 C CNN
+F 2 "adc_lib:LP5907" H 2900 1300 60  0001 C CNN
 F 3 "" H 2900 1300 60  0001 C CNN
 	1    2900 1600
@@
 L GND #PWR04
 U 1 1 59784C9E
-P 1550 3200
-F 0 "#PWR04" H 1550 2950 50  0001 C CNN
-F 1 "GND" H 1550 3050 50  0000 C CNN
-F 2 "" H 1550 3200 50  0000 C CNN
-F 3 "" H 1550 3200 50  0000 C CNN
-	1    1550 3200
+P 1650 3250
+F 0 "#PWR04" H 1650 3000 50  0001 C CNN
+F 1 "GND" H 1650 3100 50  0000 C CNN
+F 2 "" H 1650 3250 50  0000 C CNN
+F 3 "" H 1650 3250 50  0000 C CNN
+	1    1650 3250
 	1    0    0    -1
 $EndComp
@@
 F 0 "C1" H 2075 1950 50  0000 L CNN
 F 1 "1u" H 2075 1750 50  0000 L CNN
-F 2 "" H 2088 1700 50  0000 C CNN
+F 2 "adc_lib:C0603" H 2088 1700 50  0001 C CNN
 F 3 "" H 2050 1850 50  0000 C CNN
 	1    2050 1850
@@
 F 0 "C4" H 3625 1950 50  0000 L CNN
 F 1 "1u" H 3625 1750 50  0000 L CNN
-F 2 "" H 3638 1700 50  0000 C CNN
+F 2 "adc_lib:C0603" H 3638 1700 50  0001 C CNN
 F 3 "" H 3600 1850 50  0000 C CNN
 	1    3600 1850
@@
 F 0 "R1" V 4630 1500 50  0000 C CNN
 F 1 "680" V 4550 1500 50  0000 C CNN
-F 2 "" V 4480 1500 50  0000 C CNN
+F 2 "adc_lib:R0603" V 4480 1500 50  0001 C CNN
 F 3 "" H 4550 1500 50  0000 C CNN
 	1    4550 1500
@@
 F 0 "L3" V 4500 1750 50  0000 C CNN
 F 1 "8.2u" V 4625 1750 50  0000 C CNN
-F 2 "" H 4550 1750 50  0000 C CNN
+F 2 "adc_lib:L1008" H 4550 1750 50  0001 C CNN
 F 3 "" H 4550 1750 50  0000 C CNN
 	1    4550 1750
@@
 F 0 "C6" H 4225 2000 50  0000 L CNN
 F 1 "0.1u" H 4225 1800 50  0000 L CNN
-F 2 "" H 4238 1750 50  0000 C CNN
+F 2 "adc_lib:C0603" H 4238 1750 50  0001 C CNN
 F 3 "" H 4200 1900 50  0000 C CNN
 	1    4200 1900
@@
 F 0 "C8" H 5225 2000 50  0000 L CNN
 F 1 "0.1u" H 5225 1800 50  0000 L CNN
-F 2 "" H 5238 1750 50  0000 C CNN
+F 2 "adc_lib:C0603" H 5238 1750 50  0001 C CNN
 F 3 "" H 5200 1900 50  0000 C CNN
 	1    5200 1900
@@
 F 0 "L4" V 5450 1500 50  0000 C CNN
 F 1 "3.3u" V 5575 1500 50  0000 C CNN
-F 2 "" H 5500 1500 50  0000 C CNN
+F 2 "adc_lib:L0603" H 5500 1500 50  0001 C CNN
 F 3 "" H 5500 1500 50  0000 C CNN
 	1    5500 1500
@@
 F 0 "U2" H 5600 2600 60  0000 C CNN
 F 1 "PSA4-5043+" H 5150 3150 60  0000 C CNN
-F 2 "" H 5150 3150 60  0001 C CNN
+F 2 "adc_lib:MMM1362" H 5150 3150 60  0001 C CNN
 F 3 "" H 5150 3150 60  0001 C CNN
 	1    5300 2900
@@
 	1050 5000 1250 5000
 Wire Wire Line
-	1950 5000 2100 5000
-Wire Wire Line
-	2100 5000 2100 4850
+	2100 5000 1950 5000
+Wire Wire Line
+	2100 4850 2100 5000
 Wire Wire Line
 	1950 5100 2100 5100
@@
 	1050 5100 1250 5100
 Wire Wire Line
-	1750 2650 1550 2650
-Wire Wire Line
-	1550 2650 1550 3200
-Wire Wire Line
-	1750 2750 1550 2750
-Connection ~ 1550 2750
-Wire Wire Line
-	1750 2850 1550 2850
-Connection ~ 1550 2850
-Wire Wire Line
-	1750 2950 1550 2950
-Connection ~ 1550 2950
+	1850 2700 1650 2700
+Wire Wire Line
+	1650 2700 1650 3250
+Wire Wire Line
+	1850 2900 1650 2900
+Connection ~ 1650 2900
 Wire Wire Line
 	2500 1600 2400 1600
@@
 F 0 "C2" H 2775 3050 50  0000 L CNN
 F 1 "27p" H 2775 2850 50  0000 L CNN
-F 2 "" H 2788 2800 50  0000 C CNN
+F 2 "adc_lib:C0603" H 2788 2800 50  0001 C CNN
 F 3 "" H 2750 2950 50  0000 C CNN
 	1    2750 2950
@@
 F 0 "C3" H 3125 2900 50  0000 L CNN
 F 1 "12p" H 3125 2700 50  0000 L CNN
-F 2 "" H 3138 2650 50  0000 C CNN
+F 2 "adc_lib:C0603" H 3138 2650 50  0001 C CNN
 F 3 "" H 3100 2800 50  0000 C CNN
 	1    3100 2800
@@
 F 0 "L1" V 3350 2800 50  0000 C CNN
 F 1 "330n" V 3475 2800 50  0000 C CNN
-F 2 "" H 3400 2800 50  0000 C CNN
+F 2 "adc_lib:L0603" H 3400 2800 50  0001 C CNN
 F 3 "" H 3400 2800 50  0000 C CNN
 	1    3400 2800
@@
 F 0 "L2" V 3600 2950 50  0000 C CNN
 F 1 "27n" V 3725 2950 50  0000 C CNN
-F 2 "" H 3650 2950 50  0000 C CNN
+F 2 "adc_lib:L0603" H 3650 2950 50  0001 C CNN
 F 3 "" H 3650 2950 50  0000 C CNN
 	1    3650 2950
@@
 F 0 "C5" H 3975 3050 50  0000 L CNN
 F 1 "130p" H 3975 2850 50  0000 L CNN
-F 2 "" H 3988 2800 50  0000 C CNN
+F 2 "adc_lib:C0603" H 3988 2800 50  0001 C CNN
 F 3 "" H 3950 2950 50  0000 C CNN
 	1    3950 2950
@@
 F 0 "C7" H 4375 2900 50  0000 L CNN
 F 1 "0.1u" H 4375 2700 50  0000 L CNN
-F 2 "" H 4388 2650 50  0000 C CNN
+F 2 "adc_lib:C0603" H 4388 2650 50  0001 C CNN
 F 3 "" H 4350 2800 50  0000 C CNN
 	1    4350 2800
@@
 F 0 "C10" H 6725 3100 50  0000 L CNN
 F 1 "5p" H 6725 2900 50  0000 L CNN
-F 2 "" H 6738 2850 50  0000 C CNN
+F 2 "adc_lib:C0603" H 6738 2850 50  0001 C CNN
 F 3 "" H 6700 3000 50  0000 C CNN
 	1    6700 3000
@@
 F 0 "C9" H 6725 2800 50  0000 L CNN
 F 1 "9p" H 6725 2600 50  0000 L CNN
-F 2 "" H 6738 2550 50  0000 C CNN
+F 2 "adc_lib:C0603" H 6738 2550 50  0001 C CNN
 F 3 "" H 6700 2700 50  0000 C CNN
 	1    6700 2700
@@
 F 0 "L5" V 6950 3000 50  0000 C CNN
 F 1 "560n" V 7075 3000 50  0000 C CNN
-F 2 "" H 7000 3000 50  0000 C CNN
+F 2 "adc_lib:L0603" H 7000 3000 50  0001 C CNN
 F 3 "" H 7000 3000 50  0000 C CNN
 	1    7000 3000
@@
 F 0 "L6" V 7400 3150 50  0000 C CNN
 F 1 "100n" V 7525 3150 50  0000 C CNN
-F 2 "" H 7450 3150 50  0000 C CNN
+F 2 "adc_lib:L0603" H 7450 3150 50  0001 C CNN
 F 3 "" H 7450 3150 50  0000 C CNN
 	1    7450 3150
@@
 F 0 "C11" H 7475 3550 50  0000 L CNN
 F 1 "68p" H 7475 3350 50  0000 L CNN
-F 2 "" H 7488 3300 50  0000 C CNN
+F 2 "adc_lib:C0603" H 7488 3300 50  0001 C CNN
 F 3 "" H 7450 3450 50  0000 C CNN
 	1    7450 3450
@@
 F 0 "C12" H 7825 3550 50  0000 L CNN
 F 1 "100p" H 7825 3350 50  0000 L CNN
-F 2 "" H 7838 3300 50  0000 C CNN
+F 2 "adc_lib:C0603" H 7838 3300 50  0001 C CNN
 F 3 "" H 7800 3450 50  0000 C CNN
 	1    7800 3450
@@
 F 0 "L7" V 8050 3000 50  0000 C CNN
 F 1 "560n" V 8175 3000 50  0000 C CNN
-F 2 "" H 8100 3000 50  0000 C CNN
+F 2 "adc_lib:L0603" H 8100 3000 50  0001 C CNN
 F 3 "" H 8100 3000 50  0000 C CNN
 	1    8100 3000
@@
 F 0 "C13" H 8425 2850 50  0000 L CNN
 F 1 "5p" H 8425 2650 50  0000 L CNN
-F 2 "" H 8438 2600 50  0000 C CNN
+F 2 "adc_lib:C0603" H 8438 2600 50  0001 C CNN
 F 3 "" H 8400 2750 50  0000 C CNN
 	1    8400 2750
@@
 F 0 "C14" H 8425 3100 50  0000 L CNN
 F 1 "5p" H 8425 2900 50  0000 L CNN
-F 2 "" H 8438 2850 50  0000 C CNN
+F 2 "adc_lib:C0603" H 8438 2850 50  0001 C CNN
 F 3 "" H 8400 3000 50  0000 C CNN
 	1    8400 3000
@@
 L GND #PWR012
 U 1 1 597A2125
-P 9950 3350
-F 0 "#PWR012" H 9950 3100 50  0001 C CNN
-F 1 "GND" H 9950 3200 50  0000 C CNN
-F 2 "" H 9950 3350 50  0000 C CNN
-F 3 "" H 9950 3350 50  0000 C CNN
-	1    9950 3350
-	1    0    0    -1
-$EndComp
-Wire Wire Line
-	9800 3150 9950 3150
-Wire Wire Line
-	9950 2850 9950 3350
-Wire Wire Line
-	9800 3050 9950 3050
-Connection ~ 9950 3150
-Wire Wire Line
-	9800 2950 9950 2950
-Connection ~ 9950 3050
-Wire Wire Line
-	9800 2850 9950 2850
-Connection ~ 9950 2950
+P 9850 3400
+F 0 "#PWR012" H 9850 3150 50  0001 C CNN
+F 1 "GND" H 9850 3250 50  0000 C CNN
+F 2 "" H 9850 3400 50  0000 C CNN
+F 3 "" H 9850 3400 50  0000 C CNN
+	1    9850 3400
+	1    0    0    -1
+$EndComp
+Wire Wire Line
+	9850 2900 9850 3400
+Wire Wire Line
+	9700 3100 9850 3100
+Connection ~ 9850 3100
+Wire Wire Line
+	9700 2900 9850 2900
 Wire Notes Line
 	3950 1350 3950 2300
@@
 F 0 "R2" V 2430 1700 50  0000 C CNN
 F 1 "10k" V 2350 1700 50  0000 C CNN
-F 2 "" V 2280 1700 50  0000 C CNN
+F 2 "adc_lib:R0603" V 2280 1700 50  0001 C CNN
 F 3 "" H 2350 1700 50  0000 C CNN
 	1    2350 1700
@@
 Text Notes 5400 1700 0    60   ~ 0
 230mOhm
+$Comp
+L SMA_Edge CN1
+U 1 1 597C80E9
+P 2200 2800
+F 0 "CN1" H 2250 3100 60  0000 C CNN
+F 1 "SMA_Edge" H 2200 2500 60  0000 C CNN
+F 2 "adc_lib:SMA_Edge" H 2200 2800 60  0001 C CNN
+F 3 "" H 2200 2800 60  0001 C CNN
+	1    2200 2800
+	1    0    0    -1
+$EndComp
+$Comp
+L SMA_Edge CN2
+U 1 1 597C8478
+P 9350 3000
+F 0 "CN2" H 9400 3300 60  0000 C CNN
+F 1 "SMA_Edge" H 9350 2700 60  0000 C CNN
+F 2 "adc_lib:SMA_Edge" H 9350 3000 60  0001 C CNN
+F 3 "" H 9350 3000 60  0001 C CNN
+	1    9350 3000
+	-1   0    0    1
+$EndComp
 $EndSCHEMATC
