File: Sch/fm_bpf/fm_bpf.kicad_pcb (KiCad board)
At the start: 2 copper layers, 40.2 x 20.8 mm, 29 parts, among them CN1 SMA_Edge, CN2 SMA_Edge, U1 LP5907_SOT-23, U2 PSA4-5043+

Commit message: Add GND on top side
Routing:
- net GND: track 187.0 -> 212.7 mm, vias 81 -> 89
Changed lines of the file:
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@@
     (links 47)
     (no_connects 0)
-    (area 116.825 84.8 168.85 111.100002)
+    (area 118.949999 89.949999 159.250001 110.850001)
     (thickness 0.6)
     (drawings 10)
-    (tracks 273)
+    (tracks 291)
     (zones 0)
     (modules 29)
@@
   (segment (start 144.4 96.6) (end 145.46066 96.6) (width 0.25) (layer F.Cu) (net 1))
   (segment (start 145.46066 96.6) (end 146.76066 95.3) (width 0.25) (layer F.Cu) (net 1))
+  (segment (start 152.4 97.55) (end 153.35 97.55) (width 0.25) (layer F.Cu) (net 2))
+  (segment (start 153.35 97.55) (end 154.4 96.5) (width 0.25) (layer F.Cu) (net 2))
+  (via (at 154.4 96.5) (size 0.6) (drill 0.4) (layers F.Cu B.Cu) (net 2))
+  (segment (start 154.4 90.9) (end 154.4 93.9) (width 0.25) (layer F.Cu) (net 2))
+  (via (at 154.4 93.9) (size 0.6) (drill 0.4) (layers F.Cu B.Cu) (net 2))
+  (segment (start 158.2 93.9) (end 158.2 96.5) (width 0.25) (layer F.Cu) (net 2))
+  (via (at 158.2 96.5) (size 0.6) (drill 0.4) (layers F.Cu B.Cu) (net 2))
+  (segment (start 158.2 90.9) (end 158.2 93.9) (width 0.25) (layer F.Cu) (net 2))
+  (via (at 158.2 93.9) (size 0.6) (drill 0.4) (layers F.Cu B.Cu) (net 2))
+  (segment (start 154.4 90.9) (end 158.2 90.9) (width 0.25) (layer F.Cu) (net 2))
+  (via (at 158.2 90.9) (size 0.6) (drill 0.4) (layers F.Cu B.Cu) (net 2))
+  (segment (start 150.8 90.9) (end 154.4 90.9) (width 0.25) (layer F.Cu) (net 2))
+  (via (at 154.4 90.9) (size 0.6) (drill 0.4) (layers F.Cu B.Cu) (net 2))
+  (segment (start 150.8 94.9) (end 150.8 90.9) (width 0.25) (layer F.Cu) (net 2))
+  (via (at 150.8 90.9) (size 0.6) (drill 0.4) (layers F.Cu B.Cu) (net 2))
+  (segment (start 149.1 97.55) (end 149.1 96.6) (width 0.25) (layer F.Cu) (net 2))
+  (segment (start 149.1 96.6) (end 150.8 94.9) (width 0.25) (layer F.Cu) (net 2))
+  (via (at 150.8 94.9) (size 0.6) (drill 0.4) (layers F.Cu B.Cu) (net 2))
   (segment (start 136.85 97.65) (end 136.85 95.9) (width 0.25) (layer F.Cu) (net 2))
   (segment (start 136.85 95.9) (end 137 95.75) (width 0.25) (layer F.Cu) (net 2))
@@
     (polygon
       (pts
-        (xy 142.3 93) (xy 142.3 94) (xy 143.2 94.8) (xy 143.2 97.7) (xy 145.6 97.7)
-        (xy 145.6 93)
+        (xy 142.3 93.1) (xy 142.3 94) (xy 143.2 94.8) (xy 143.2 97.7) (xy 145.6 97.7)
+        (xy 145.6 93.1)
       )
     )
@@
   )
   (zone (net 2) (net_name GND) (layer F.Cu) (hatch edge 0.508)
-    (connect_pads yes (clearance 0.2))
+    (connect_pads yes (clearance 0.3))
     (min_thickness 0.254)
     (fill yes (arc_segments 16) (thermal_gap 0.508) (thermal_bridge_width 0.508))
@@
       (pts
         (xy 141 99.6) (xy 141 101.6) (xy 147.5 101.6) (xy 148.9 100.3) (xy 152.7 100.3)
-        (xy 155.2 99.3) (xy 155.2 97.1) (xy 146.1 97.1) (xy 146.1 98) (xy 141.6 98)
-        (xy 141.6 99.6)
+        (xy 155.2 99.3) (xy 158.8 99.2) (xy 158.8 90.3) (xy 150.3 90.3) (xy 150.3 94.6)
+        (xy 146.1 97.1) (xy 146.1 98) (xy 141.6 98) (xy 141.6 99.6)
       )
     )

Commit message: Fix BOM for BPF and layout
Connections:
- CN1 pad 1: GND -> Net-(C2-Pad1)
- CN1 pad 2: Net-(C2-Pad1) -> GND
- CN2 pad 1: GND -> Net-(C13-Pad1)
- CN2 pad 2: Net-(C13-Pad1) -> GND
- U1 pad 4: Net-(U1-Pad4) -> (no net)
Other:
- board text added: "FM BPF 76-95MHz"

Commit message: BPF perhaps final
Routing:
- net Net-(C13-Pad1): track 8.23 -> 7.43 mm
Changed lines of the file:
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@@
     (thickness 0.6)
     (drawings 11)
-    (tracks 291)
+    (tracks 290)
     (zones 0)
     (modules 29)
@@
     (31 B.Cu signal)
     (33 F.Adhes user)
+    (34 B.Paste user)
     (35 F.Paste user)
+    (36 B.SilkS user)
     (37 F.SilkS user)
+    (38 B.Mask user)
     (39 F.Mask user)
     (40 Dwgs.User user)
@@
     (pad_drill 0.6)
     (pad_to_mask_clearance 0)
-    (aux_axis_origin 119 90)
+    (aux_axis_origin 119 110.8)
     (visible_elements 7FFFFFFF)
     (pcbplotparams
-      (layerselection 0x00030_80000001)
+      (layerselection 0x010fe_80000001)
       (usegerberextensions false)
       (excludeedgelayer true)
@@
       (outputformat 1)
       (mirror false)
-      (drillshape 1)
+      (drillshape 0)
       (scaleselection 1)
       (outputdirectory ""))
@@
   (module adc_lib:MMM1362 (layer F.Cu)
     (at 137.86 103.67 180)
-    (fp_text reference U2 (at -0.04 -2.63 180) (layer F.SilkS)
+    (fp_text reference U2 (at -0.04 -3.03 180) (layer F.SilkS)
       (effects (font (size 1 1) (thickness 0.15)))
     )
@@
   (module adc_lib:LP5907 (layer F.Cu)
     (at 141.617343 92.495056 90)
-    (fp_text reference U1 (at -0.004944 -2.717343 90) (layer F.SilkS)
+    (fp_text reference U1 (at -0.004944 -4.717343 90) (layer F.SilkS)
       (effects (font (size 1 1) (thickness 0.15)))
     )
@@
   (module adc_lib:L0603 (layer F.Cu)
     (at 145.86 103.34 90)
-    (fp_text reference L6 (at 2.14 -0.16 90) (layer F.SilkS)
+    (fp_text reference L6 (at 3.04 -0.26 90) (layer F.SilkS)
       (effects (font (size 1 1) (thickness 0.15)))
     )
@@
   (module adc_lib:L0603 (layer F.Cu)
     (at 144.03 102.64 180)
-    (fp_text reference L5 (at 0.09 1.3 180) (layer F.SilkS)
+    (fp_text reference L5 (at 0.13 2.24 180) (layer F.SilkS)
       (effects (font (size 1 1) (thickness 0.15)))
     )
@@
   (module adc_lib:L0603 (layer F.Cu)
     (at 140 101.9 90)
-    (fp_text reference L4 (at 0.8 1.3 90) (layer F.SilkS)
+    (fp_text reference L4 (at 1.3 1.6 90) (layer F.SilkS)
       (effects (font (size 1 1) (thickness 0.15)))
     )
@@
   (module adc_lib:L0603 (layer F.Cu)
     (at 132.95 105.61 90)
-    (fp_text reference L2 (at 2.11 0.05 90) (layer F.SilkS)
+    (fp_text reference L2 (at -2.09 -0.15 90) (layer F.SilkS)
       (effects (font (size 1 1) (thickness 0.15)))
     )
@@
   (module adc_lib:L0603 (layer F.Cu)
     (at 131.29 104.82 180)
-    (fp_text reference L1 (at 0.09 1.3 180) (layer F.SilkS)
+    (fp_text reference L1 (at -0.11 2.62 180) (layer F.SilkS)
       (effects (font (size 1 1) (thickness 0.15)))
     )
@@
       (net 4 "Net-(C3-Pad1)"))
   )
-  (module adc_lib:SMA_Edge (layer F.Cu)
-    (at 156.66 102.63 270)
-    (fp_text reference CN2 (at 5.57 3.76 270) (layer F.SilkS)
-      (effects (font (size 1 1) (thickness 0.15)))
-    )
-    (fp_text value SMA_Edge (at -4.8 3.8 270) (layer F.Fab)
-      (effects (font (size 1 1) (thickness 0.15)))
-    )
-    (pad 2 connect rect (at -4.318 0 270) (size 2.4 5.08) (layers F.Cu F.Mask)
-      (net 2 GND))
-    (pad 3 connect rect (at 4.318 0 270) (size 2.4 5.08) (layers F.Cu F.Mask)
-      (net 2 GND))
-    (pad 1 connect rect (at 0 0 270) (size 2.286 5.08) (layers F.Cu F.Mask)
-      (net 13 "Net-(C13-Pad1)"))
-    (pad 4 connect rect (at -4.318 0 270) (size 2.4 5.08) (layers B.Cu)
-      (net 2 GND))
-    (pad 5 connect rect (at 4.318 0 270) (size 2.4 5.08) (layers B.Cu)
-      (net 2 GND))
-  )
-  (module adc_lib:SMA_Edge (layer F.Cu)
-    (at 121.6 104.82 270)
-    (fp_text reference CN1 (at 4.08 -3.7 270) (layer F.SilkS)
-      (effects (font (size 1 1) (thickness 0.15)))
-    )
-    (fp_text value SMA_Edge (at -4.8 3.8 270) (layer F.Fab)
-      (effects (font (size 1 1) (thickness 0.15)))
-    )
-    (pad 2 connect rect (at -4.318 0 270) (size 2.4 5.08) (layers F.Cu F.Mask)
-      (net 2 GND))
-    (pad 3 connect rect (at 4.318 0 270) (size 2.4 5.08) (layers F.Cu F.Mask)
-      (net 2 GND))
-    (pad 1 connect rect (at 0 0 270) (size 2.286 5.08) (layers F.Cu F.Mask)
-      (net 3 "Net-(C2-Pad1)"))
-    (pad 4 connect rect (at -4.318 0 270) (size 2.4 5.08) (layers B.Cu)
-      (net 2 GND))
-    (pad 5 connect rect (at 4.318 0 270) (size 2.4 5.08) (layers B.Cu)
-      (net 2 GND))
-  )
   (module adc_lib:C0603 (layer F.Cu)
     (at 152 102.64 180)
-    (fp_text reference C14 (at -0.1 -1.36 180) (layer F.SilkS)
+    (fp_text reference C14 (at -0.1 -2.86 180) (layer F.SilkS)
       (effects (font (size 1 1) (thickness 0.15)))
     )
@@
   (module adc_lib:C0603 (layer F.Cu)
     (at 150.1 101.5 180)
-    (fp_text reference C13 (at -0.05 1.55 180) (layer F.SilkS)
+    (fp_text reference C13 (at -0.05 2 180) (layer F.SilkS)
       (effects (font (size 1 1) (thickness 0.15)))
     )
@@
   (module adc_lib:C0603 (layer F.Cu)
     (at 147.06 103.34 90)
-    (fp_text reference C12 (at 2.74 -0.06 90) (layer F.SilkS)
+    (fp_text reference C12 (at 3.44 -0.06 90) (layer F.SilkS)
       (effects (font (size 1 1) (thickness 0.15)))
     )
@@
   (module adc_lib:C0603 (layer F.Cu)
     (at 146.56 105.04 180)
-    (fp_text reference C11 (at 0.06 -1.36 180) (layer F.SilkS)
+    (fp_text reference C11 (at 0.06 -1.96 180) (layer F.SilkS)
       (effects (font (size 1 1) (thickness 0.15)))
     )
@@
   (module adc_lib:C0603 (layer F.Cu)
     (at 141.54 102.64 180)
-    (fp_text reference C10 (at 1.24 -1.66 180) (layer F.SilkS)
+    (fp_text reference C10 (at 0.24 -3.46 180) (layer F.SilkS)
       (effects (font (size 1 1) (thickness 0.15)))
     )
@@
   (module adc_lib:C0603 (layer F.Cu)
     (at 142.8 103.8 180)
-    (fp_text reference C9 (at 0.1 -1.3 180) (layer F.SilkS)
+    (fp_text reference C9 (at 0.1 -3.7 180) (layer F.SilkS)
       (effects (font (size 1 1) (thickness 0.15)))
     )
@@
   (module adc_lib:C0603 (layer F.Cu)
     (at 139.3 99.9 180)
-    (fp_text reference C8 (at 2.4 0.3 180) (layer F.SilkS)
+    (fp_text reference C8 (at 3 0 180) (layer F.SilkS)
       (effects (font (size 1 1) (thickness 0.15)))
     )
@@
   (module adc_lib:C0603 (layer F.Cu)
     (at 135.66 104.82)
-    (fp_text reference C7 (at 0.04 1.38) (layer F.SilkS)
+    (fp_text reference C7 (at 0.24 2.78) (layer F.SilkS)
       (effects (font (size 1 1) (thickness 0.15)))
     )
@@
   (module adc_lib:C0603 (layer F.Cu)
     (at 134.01 105.55 90)
-    (fp_text reference C5 (at 2.05 0.29 90) (layer F.SilkS)
+    (fp_text reference C5 (at -2.35 0.29 90) (layer F.SilkS)
       (effects (font (size 1 1) (thickness 0.15)))
     )
@@
   (module adc_lib:C0603 (layer F.Cu)
     (at 128.86 104.82 180)
-    (fp_text reference C3 (at 0.16 1.42 180) (layer F.SilkS)
+    (fp_text reference C3 (at 0.06 2.52 180) (layer F.SilkS)
       (effects (font (size 1 1) (thickness 0.15)))
     )
@@
   (module adc_lib:C0603 (layer F.Cu)
     (at 126.74 105.52 270)
-    (fp_text reference C2 (at -2.12 0.24 360) (layer F.SilkS)
+    (fp_text reference C2 (at -3.22 0.14 360) (layer F.SilkS)
       (effects (font (size 1 1) (thickness 0.15)))
     )
@@
       (net 1 +5V))
     (pad 2 smd rect (at 0.7 0 90) (size 0.7 0.8) (layers F.Cu F.Paste F.Mask)
+      (net 2 GND))
+  )
+  (module adc_lib:SMA_Edge (layer F.Cu)
+    (at 121.6 104.82 270)
+    (fp_text reference CN1 (at -7.92 0.2 270) (layer F.SilkS)
+      (effects (font (size 1 1) (thickness 0.15)))
+    )
+    (fp_text value SMA_Edge (at -4.8 3.8 270) (layer F.Fab)
+      (effects (font (size 1 1) (thickness 0.15)))
+    )
+    (pad 2 connect rect (at -4.318 0 270) (size 2.4 5.08) (layers F.Cu F.Mask)
+      (net 2 GND))
+    (pad 3 connect rect (at 4.318 0 270) (size 2.4 5.08) (layers F.Cu F.Mask)
+      (net 2 GND))
+    (pad 1 connect rect (at 0 0 270) (size 2.286 5.08) (layers F.Cu F.Mask)
+      (net 3 "Net-(C2-Pad1)"))
+    (pad 4 connect rect (at -4.318 0 270) (size 2.4 5.08) (layers B.Cu B.Mask)
+      (net 2 GND))
+    (pad 5 connect rect (at 4.318 0 270) (size 2.4 5.08) (layers B.Cu B.Mask)
+      (net 2 GND))
+  )
+  (module adc_lib:SMA_Edge (layer F.Cu)
+    (at 156.66 102.63 270)
+    (fp_text reference CN2 (at 4.3 4 270) (layer F.SilkS)
+      (effects (font (size 1 1) (thickness 0.15)))
+    )
+    (fp_text value SMA_Edge (at -4.8 3.8 270) (layer F.Fab)
+      (effects (font (size 1 1) (thickness 0.15)))
+    )
+    (pad 2 connect rect (at -4.318 0 270) (size 2.4 5.08) (layers F.Cu F.Mask)
+      (net 2 GND))
+    (pad 3 connect rect (at 4.318 0 270) (size 2.4 5.08) (layers F.Cu F.Mask)
+      (net 2 GND))
+    (pad 1 connect rect (at 0 0 270) (size 2.286 5.08) (layers F.Cu F.Mask)
+      (net 13 "Net-(C13-Pad1)"))
+    (pad 4 connect rect (at -4.318 0 270) (size 2.4 5.08) (layers B.Cu B.Mask)
+      (net 2 GND))
+    (pad 5 connect rect (at 4.318 0 270) (size 2.4 5.08) (layers B.Cu B.Mask)
       (net 2 GND))
   )
@@
   (segment (start 156.65 102.64) (end 156.66 102.63) (width 0.25) (layer F.Cu) (net 13))
   (segment (start 156.64 102.65) (end 156.66 102.63) (width 0.8) (layer F.Cu) (net 13))
-  (segment (start 156.09 103.2) (end 156.66 102.63) (width 0.8) (layer F.Cu) (net 13))
   (segment (start 152.7 102.64) (end 156.65 102.64) (width 0.25) (layer F.Cu) (net 13))
   (segment (start 150.8 101.5) (end 151.56 101.5) (width 0.25) (layer F.Cu) (net 13))
