File: Sch/fm_bpf/fm_bpf.kicad_pcb (KiCad board)
At the start: 2 copper layers, 40.2 x 20.8 mm, 29 parts, among them CN1 SMA_Edge, CN2 SMA_Edge, U1 LP5907_SOT-23, U2 PSA4-5043+

Commit message: Add revision marking to BPF
Other:
- board text added: "FM BPF rev 0.1 76-95MHz"
- board text removed: "FM BPF 76-95MHz"
Changed lines of the file:
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@@
     (links 51)
     (no_connects 0)
-    (area 116.825 84.8 168.85 110.900002)
+    (area 118.949999 89.949999 159.250001 110.850001)
     (thickness 0.6)
     (drawings 11)
@@
       (psa4output false)
       (plotreference true)
-      (plotvalue true)
+      (plotvalue false)
       (plotinvisibletext false)
       (padsonsilk false)
@@
       (net 2 GND))
   )
-  (gr_text "FM BPF\n76-95MHz" (at 130.9 97.6) (layer B.SilkS)
+  (gr_text "FM BPF rev 0.1\n76-95MHz" (at 130 95.8) (layer B.SilkS)
     (effects (font (size 1.5 1.5) (thickness 0.3)) (justify mirror))
   )

Commit message: Improve layout
Routing:
- net GND: track 212.7 -> 238.5 mm, vias 89 -> 91
Changed lines of the file:
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@@
     (links 51)
     (no_connects 0)
-    (area 118.949999 89.949999 159.250001 110.850001)
+    (area 116.825 84.8 168.85 110.900002)
     (thickness 0.6)
     (drawings 11)
-    (tracks 290)
+    (tracks 307)
     (zones 0)
     (modules 29)
@@
   (segment (start 144.4 96.6) (end 145.46066 96.6) (width 0.25) (layer F.Cu) (net 1))
   (segment (start 145.46066 96.6) (end 146.76066 95.3) (width 0.25) (layer F.Cu) (net 1))
+  (segment (start 133 95.1) (end 133 99.6) (width 0.25) (layer F.Cu) (net 2))
+  (via (at 133 99.6) (size 0.6) (drill 0.4) (layers F.Cu B.Cu) (net 2))
+  (segment (start 128.3 95.1) (end 133 95.1) (width 0.25) (layer F.Cu) (net 2))
+  (via (at 133 95.1) (size 0.6) (drill 0.4) (layers F.Cu B.Cu) (net 2))
+  (segment (start 128.3 99.6) (end 128.3 99) (width 0.25) (layer F.Cu) (net 2))
+  (segment (start 128.3 99) (end 124.4 95.1) (width 0.25) (layer F.Cu) (net 2))
+  (via (at 124.4 95.1) (size 0.6) (drill 0.4) (layers F.Cu B.Cu) (net 2))
+  (segment (start 128.3 95.1) (end 128.3 99.6) (width 0.25) (layer F.Cu) (net 2))
+  (via (at 128.3 99.6) (size 0.6) (drill 0.4) (layers F.Cu B.Cu) (net 2))
+  (segment (start 128.35 90.7) (end 128.35 95.05) (width 0.25) (layer F.Cu) (net 2))
+  (segment (start 128.35 95.05) (end 128.3 95.1) (width 0.25) (layer F.Cu) (net 2))
+  (via (at 128.3 95.1) (size 0.6) (drill 0.4) (layers F.Cu B.Cu) (net 2))
+  (segment (start 125.5 106.7) (end 124.9 106.7) (width 0.25) (layer F.Cu) (net 2))
+  (segment (start 124.9 106.7) (end 124.2 107.4) (width 0.25) (layer F.Cu) (net 2))
+  (via (at 124.2 107.4) (size 0.6) (drill 0.4) (layers F.Cu B.Cu) (net 2))
+  (segment (start 126.74 106.22) (end 125.98 106.22) (width 0.25) (layer F.Cu) (net 2))
+  (segment (start 125.98 106.22) (end 125.5 106.7) (width 0.25) (layer F.Cu) (net 2))
+  (via (at 125.5 106.7) (size 0.6) (drill 0.4) (layers F.Cu B.Cu) (net 2))
+  (segment (start 131.2 106.4) (end 128.8 106.4) (width 0.25) (layer F.Cu) (net 2))
+  (segment (start 128.8 106.4) (end 128.7 106.3) (width 0.25) (layer F.Cu) (net 2))
+  (via (at 128.7 106.3) (size 0.6) (drill 0.4) (layers F.Cu B.Cu) (net 2))
+  (segment (start 132.95 106.31) (end 131.29 106.31) (width 0.25) (layer F.Cu) (net 2))
+  (segment (start 131.29 106.31) (end 131.2 106.4) (width 0.25) (layer F.Cu) (net 2))
+  (via (at 131.2 106.4) (size 0.6) (drill 0.4) (layers F.Cu B.Cu) (net 2))
+  (segment (start 135.7 106.4) (end 138.4 106.4) (width 0.25) (layer F.Cu) (net 2))
+  (via (at 138.4 106.4) (size 0.6) (drill 0.4) (layers F.Cu B.Cu) (net 2))
+  (segment (start 134.01 106.25) (end 135.55 106.25) (width 0.25) (layer F.Cu) (net 2))
+  (segment (start 135.55 106.25) (end 135.7 106.4) (width 0.25) (layer F.Cu) (net 2))
+  (via (at 135.7 106.4) (size 0.6) (drill 0.4) (layers F.Cu B.Cu) (net 2))
+  (segment (start 145.1 106.3) (end 144.8 106.3) (width 0.25) (layer F.Cu) (net 2))
+  (segment (start 144.8 106.3) (end 143.9 105.4) (width 0.25) (layer F.Cu) (net 2))
+  (via (at 143.9 105.4) (size 0.6) (drill 0.4) (layers F.Cu B.Cu) (net 2))
+  (segment (start 146.9 106.4) (end 145.2 106.4) (width 0.25) (layer F.Cu) (net 2))
+  (via (at 145.1 106.3) (size 0.6) (drill 0.4) (layers F.Cu B.Cu) (net 2))
+  (segment (start 145.2 106.4) (end 145.1 106.3) (width 0.25) (layer F.Cu) (net 2))
+  (segment (start 146.2 106.5) (end 145.6 106.5) (width 0.25) (layer F.Cu) (net 2))
+  (segment (start 145.6 106.5) (end 145 106.5) (width 0.25) (layer F.Cu) (net 2))
+  (segment (start 146.9 106.4) (end 146.475736 106.4) (width 0.25) (layer F.Cu) (net 2))
+  (segment (start 146.475736 106.4) (end 146.375736 106.5) (width 0.25) (layer F.Cu) (net 2))
+  (segment (start 146.375736 106.5) (end 145.6 106.5) (width 0.25) (layer F.Cu) (net 2))
+  (segment (start 147.26 105.04) (end 147.26 106.04) (width 0.25) (layer F.Cu) (net 2))
+  (segment (start 147.26 106.04) (end 146.9 106.4) (width 0.25) (layer F.Cu) (net 2))
+  (via (at 146.9 106.4) (size 0.6) (drill 0.4) (layers F.Cu B.Cu) (net 2))
+  (segment (start 142.8 105.4) (end 140.9 105.4) (width 0.25) (layer F.Cu) (net 2))
+  (segment (start 140.9 105.4) (end 140.5 105) (width 0.25) (layer F.Cu) (net 2))
+  (via (at 140.5 105) (size 0.6) (drill 0.4) (layers F.Cu B.Cu) (net 2))
+  (segment (start 144.4 105.9) (end 143.3 105.9) (width 0.25) (layer F.Cu) (net 2))
+  (segment (start 143.3 105.9) (end 142.8 105.4) (width 0.25) (layer F.Cu) (net 2))
+  (segment (start 145 106.5) (end 144.4 105.9) (width 0.25) (layer F.Cu) (net 2))
+  (segment (start 147.26 105.04) (end 147.26 105.44) (width 0.25) (layer F.Cu) (net 2))
+  (segment (start 147.26 105.44) (end 146.2 106.5) (width 0.25) (layer F.Cu) (net 2))
+  (segment (start 151 104.2) (end 148.2 104.2) (width 0.25) (layer F.Cu) (net 2))
+  (via (at 148.2 104.2) (size 0.6) (drill 0.4) (layers F.Cu B.Cu) (net 2))
+  (segment (start 152.3 104.95) (end 151.75 104.95) (width 0.25) (layer F.Cu) (net 2))
+  (segment (start 151.75 104.95) (end 151 104.2) (width 0.25) (layer F.Cu) (net 2))
+  (via (at 151 104.2) (size 0.6) (drill 0.4) (layers F.Cu B.Cu) (net 2))
   (segment (start 136.85 97.65) (end 136.85 95.9) (width 0.25) (layer F.Cu) (net 2))
   (segment (start 136.85 95.9) (end 137 95.75) (width 0.25) (layer F.Cu) (net 2))
@@
   (segment (start 124.45 109.348) (end 124.45 110.3) (width 0.25) (layer F.Cu) (net 2))
   (via (at 124.45 110.1) (size 0.6) (drill 0.4) (layers F.Cu B.Cu) (net 2))
-  (segment (start 125.55 106.65) (end 124.9 106.65) (width 0.25) (layer F.Cu) (net 2))
-  (segment (start 124.9 106.65) (end 124.2 107.35) (width 0.25) (layer F.Cu) (net 2))
-  (via (at 124.2 107.35) (size 0.6) (drill 0.4) (layers F.Cu B.Cu) (net 2))
-  (segment (start 127.7 106.35) (end 125.85 106.35) (width 0.25) (layer B.Cu) (net 2))
-  (segment (start 125.85 106.35) (end 125.55 106.65) (width 0.25) (layer B.Cu) (net 2))
-  (via (at 125.55 106.65) (size 0.6) (drill 0.4) (layers F.Cu B.Cu) (net 2))
-  (segment (start 129.45 106.35) (end 127.7 106.35) (width 0.25) (layer F.Cu) (net 2))
-  (via (at 127.7 106.35) (size 0.6) (drill 0.4) (layers F.Cu B.Cu) (net 2))
-  (segment (start 131.75 106.35) (end 129.45 106.35) (width 0.25) (layer B.Cu) (net 2))
-  (via (at 129.45 106.35) (size 0.6) (drill 0.4) (layers F.Cu B.Cu) (net 2))
-  (segment (start 135 106.45) (end 131.85 106.45) (width 0.25) (layer F.Cu) (net 2))
-  (segment (start 131.85 106.45) (end 131.75 106.35) (width 0.25) (layer F.Cu) (net 2))
-  (via (at 131.75 106.35) (size 0.6) (drill 0.4) (layers F.Cu B.Cu) (net 2))
-  (segment (start 136.5 106.45) (end 135 106.45) (width 0.25) (layer B.Cu) (net 2))
-  (via (at 135 106.45) (size 0.6) (drill 0.4) (layers F.Cu B.Cu) (net 2))
-  (segment (start 138.45 106.4) (end 136.55 106.4) (width 0.25) (layer F.Cu) (net 2))
-  (segment (start 136.55 106.4) (end 136.5 106.45) (width 0.25) (layer F.Cu) (net 2))
-  (via (at 136.5 106.45) (size 0.6) (drill 0.4) (layers F.Cu B.Cu) (net 2))
-  (segment (start 140.45 105.05) (end 139.8 105.05) (width 0.25) (layer B.Cu) (net 2))
-  (segment (start 139.8 105.05) (end 138.45 106.4) (width 0.25) (layer B.Cu) (net 2))
-  (via (at 138.45 106.4) (size 0.6) (drill 0.4) (layers F.Cu B.Cu) (net 2))
-  (segment (start 142.8 105.4) (end 140.8 105.4) (width 0.25) (layer F.Cu) (net 2))
-  (segment (start 140.8 105.4) (end 140.45 105.05) (width 0.25) (layer F.Cu) (net 2))
-  (via (at 140.45 105.05) (size 0.6) (drill 0.4) (layers F.Cu B.Cu) (net 2))
-  (segment (start 144.4 105.9) (end 143.3 105.9) (width 0.25) (layer B.Cu) (net 2))
-  (segment (start 143.3 105.9) (end 142.8 105.4) (width 0.25) (layer B.Cu) (net 2))
-  (via (at 142.8 105.4) (size 0.6) (drill 0.4) (layers F.Cu B.Cu) (net 2))
-  (segment (start 146.15 106.5) (end 145 106.5) (width 0.25) (layer F.Cu) (net 2))
-  (segment (start 145 106.5) (end 144.4 105.9) (width 0.25) (layer F.Cu) (net 2))
-  (via (at 144.4 105.9) (size 0.6) (drill 0.4) (layers F.Cu B.Cu) (net 2))
-  (segment (start 148 104.25) (end 146.15 106.1) (width 0.25) (layer B.Cu) (net 2))
-  (segment (start 146.15 106.1) (end 146.15 106.5) (width 0.25) (layer B.Cu) (net 2))
-  (via (at 146.15 106.5) (size 0.6) (drill 0.4) (layers F.Cu B.Cu) (net 2))
-  (segment (start 149.2 104.25) (end 148 104.25) (width 0.25) (layer F.Cu) (net 2))
-  (via (at 148 104.25) (size 0.6) (drill 0.4) (layers F.Cu B.Cu) (net 2))
-  (segment (start 150.35 104.75) (end 149.7 104.75) (width 0.25) (layer B.Cu) (net 2))
-  (segment (start 149.7 104.75) (end 149.2 104.25) (width 0.25) (layer B.Cu) (net 2))
-  (via (at 149.2 104.25) (size 0.6) (drill 0.4) (layers F.Cu B.Cu) (net 2))
   (segment (start 152.3 104.95) (end 150.55 104.95) (width 0.25) (layer F.Cu) (net 2))
   (segment (start 150.55 104.95) (end 150.35 104.75) (width 0.25) (layer F.Cu) (net 2))
-  (via (at 150.35 104.75) (size 0.6) (drill 0.4) (layers F.Cu B.Cu) (net 2))
   (segment (start 153.5 105.7) (end 153.05 105.7) (width 0.25) (layer B.Cu) (net 2))
   (segment (start 153.05 105.7) (end 152.3 104.95) (width 0.25) (layer B.Cu) (net 2))
@@
         (xy 137.8 102.433333) (xy 138 103.3) (xy 138.35 103.8) (xy 138.8 104.3) (xy 140.6 104.3)
         (xy 141.3 104.9) (xy 144.1 104.9) (xy 145.3 105.9) (xy 146.6 105.9) (xy 146.6 103.7)
-        (xy 149.9 103.7) (xy 150.9 104.4) (xy 152.6 104.4) (xy 153.8 105.2) (xy 154.6 105.8)
+        (xy 149.9 103.7) (xy 151.2 103.7) (xy 152.6 104.4) (xy 153.8 105.2) (xy 154.6 105.8)
         (xy 159 107.6) (xy 159 110.7) (xy 119.1 110.7) (xy 119.1 108.2) (xy 122.2 108)
         (xy 125.8 105.9) (xy 138 105.9) (xy 138 104.45) (xy 137.5 103.7) (xy 125.7 103.7)
